Commit message: fixes

File: ric_gazebo/models/komodo.xacro (robot description, xacro)
@@ -2,5 +2,5 @@
 <robot xmlns:xacro="http://www.ros.org/wiki/ric" name="ric_description">
   <link
-    name="komodo_$(arg komodo_id)_base_link">
+    name="base_link">
     <inertial>
       <origin
@@ -42,5 +42,5 @@
   </link>
   <link
-    name="komodo_$(arg komodo_id)_FR_Wheel_link">
+    name="FR_Wheel_link">
     <inertial>
       <origin
@@ -82,13 +82,13 @@
   </link>
   <joint
-    name="komodo_$(arg komodo_id)_FR_Wheel_joint"
-    type="fixed">
+    name="FR_Wheel_joint"
+    type="continuous">
     <origin
       xyz="0.165 -0.18938 0"
       rpy="-2.4325E-31 -1.9723E-15 -1.5708" />
     <parent
-      link="komodo_$(arg komodo_id)_base_link" />
-    <child
-      link="komodo_$(arg komodo_id)_FR_Wheel_link" />
+      link="base_link" />
+    <child
+      link="FR_Wheel_link" />
     <axis
       xyz="-1 0 0" />
@@ -98,5 +98,5 @@
   </joint>
   <link
-    name="komodo_$(arg komodo_id)_FL_Wheel_link">
+    name="FL_Wheel_link">
     <inertial>
       <origin
@@ -138,13 +138,13 @@
   </link>
   <joint
-    name="komodo_$(arg komodo_id)_FL_Wheel_joint"
-    type="fixed">
+    name="FL_Wheel_joint"
+    type="continuous">
     <origin
       xyz="0.165 0.18938 0"
       rpy="2.4325E-31 1.9723E-15 1.5708" />
     <parent
-      link="komodo_$(arg komodo_id)_base_link" />
-    <child
-      link="komodo_$(arg komodo_id)_FL_Wheel_link" />
+      link="base_link" />
+    <child
+      link="FL_Wheel_link" />
     <axis
       xyz="1 0 0" />
@@ -154,5 +154,5 @@
   </joint>
   <link
-    name="komodo_$(arg komodo_id)_RR_Wheel_link">
+    name="RR_Wheel_link">
     <inertial>
       <origin
@@ -194,13 +194,13 @@
   </link>
   <joint
-    name="komodo_$(arg komodo_id)_RR_Wheel_joint"
-    type="fixed">
+    name="RR_Wheel_joint"
+    type="continuous">
     <origin
       xyz="-0.165 -0.18938 0"
       rpy="-2.4325E-31 -1.9723E-15 -1.5708" />
     <parent
-      link="komodo_$(arg komodo_id)_base_link" />
-    <child
-      link="komodo_$(arg komodo_id)_RR_Wheel_link" />
+      link="base_link" />
+    <child
+      link="RR_Wheel_link" />
     <axis
       xyz="-1 0 0" />
@@ -210,5 +210,5 @@
   </joint>
   <link
-    name="komodo_$(arg komodo_id)_RL_Wheel_link">
+    name="RL_Wheel_link">
     <inertial>
       <origin
@@ -250,13 +250,13 @@
   </link>
   <joint
-    name="komodo_$(arg komodo_id)_RL_Wheel_joint"
-    type="fixed">
+    name="RL_Wheel_joint"
+    type="continuous">
     <origin
       xyz="-0.165 0.18938 0"
       rpy="2.4325E-31 1.9723E-15 1.5708" />
     <parent
-      link="komodo_$(arg komodo_id)_base_link" />
-    <child
-      link="komodo_$(arg komodo_id)_RL_Wheel_link" />
+      link="base_link" />
+    <child
+      link="RL_Wheel_link" />
     <axis
       xyz="1 0 0" />
@@ -266,5 +266,5 @@
   </joint>
   <link
-    name="komodo_$(arg komodo_id)_Left_URF_link">
+    name="Left_URF_link">
     <inertial>
       <origin
@@ -306,5 +306,5 @@
   </link>
   <joint
-    name="komodo_$(arg komodo_id)_Left_US_joint"
+    name="Left_US_joint"
     type="fixed">
     <origin
@@ -312,12 +312,12 @@
       rpy="2.4325E-31 1.9723E-15 1.5708" />
     <parent
-      link="komodo_$(arg komodo_id)_base_link" />
-    <child
-      link="komodo_$(arg komodo_id)_Left_URF_link" />
+      link="base_link" />
+    <child
+      link="Left_URF_link" />
     <axis
       xyz="0 0 0" />
   </joint>
   <link
-    name="komodo_$(arg komodo_id)_Rear_URF_link">
+    name="Rear_URF_link">
     <inertial>
       <origin
@@ -359,5 +359,5 @@
   </link>
   <joint
-    name="komodo_$(arg komodo_id)_Back_US_joint"
+    name="Back_US_joint"
     type="fixed">
     <origin
@@ -365,12 +365,12 @@
       rpy="1.9723E-15 -2.736E-15 3.1416" />
     <parent
-      link="komodo_$(arg komodo_id)_base_link" />
-    <child
-      link="komodo_$(arg komodo_id)_Rear_URF_link" />
+      link="base_link" />
+    <child
+      link="Rear_URF_link" />
     <axis
       xyz="0 0 0" />
   </joint>
   <link
-    name="komodo_$(arg komodo_id)_Right_URF_link">
+    name="Right_URF_link">
     <inertial>
       <origin
@@ -412,5 +412,5 @@
   </link>
   <joint
-    name="komodo_$(arg komodo_id)_Right_US_joint"
+    name="Right_US_joint"
     type="fixed">
     <origin
@@ -418,12 +418,12 @@
       rpy="-1.2406E-16 -1.9723E-15 -1.5708" />
     <parent
-      link="komodo_$(arg komodo_id)_base_link" />
-    <child
-      link="komodo_$(arg komodo_id)_Right_URF_link" />
+      link="base_link" />
+    <child
+      link="Right_URF_link" />
     <axis
       xyz="0 0 0" />
   </joint>
   <link
-    name="komodo_$(arg komodo_id)_Front_Camera_link">
+    name="Front_Camera_link">
     <inertial>
       <origin
@@ -465,5 +465,5 @@
   </link>
   <joint
-    name="komodo_$(arg komodo_id)_Front_Camera_joint"
+    name="Front_Camera_joint"
     type="fixed">
     <origin
@@ -471,12 +471,12 @@
       rpy="-1.5708 -1.9723E-15 -1.5708" />
     <parent
-      link="komodo_$(arg komodo_id)_base_link" />
-    <child
-      link="komodo_$(arg komodo_id)_Front_Camera_link" />
+      link="base_link" />
+    <child
+      link="Front_Camera_link" />
     <axis
       xyz="0 0 0" />
   </joint>
   <link
-    name="komodo_$(arg komodo_id)_Laser_link">
+    name="Laser_link">
     <inertial>
       <origin
@@ -518,5 +518,5 @@
   </link>
   <joint
-    name="komodo_$(arg komodo_id)_Laser_joint"
+    name="Laser_joint"
     type="fixed">
     <origin
@@ -524,12 +524,12 @@
       rpy="-1.9723E-15 2.4325E-31 0" />
     <parent
-      link="komodo_$(arg komodo_id)_base_link" />
-    <child
-      link="komodo_$(arg komodo_id)_Laser_link" />
+      link="base_link" />
+    <child
+      link="Laser_link" />
     <axis
       xyz="0 0 0" />
   </joint>
   <link
-    name="komodo_$(arg komodo_id)_Asus_Camera_link">
+    name="Asus_Camera_link">
     <inertial>
       <origin
@@ -571,5 +571,5 @@
   </link>
   <joint
-    name="komodo_$(arg komodo_id)_Asus_joint"
+    name="Asus_joint"
     type="fixed">
     <origin
@@ -577,12 +577,12 @@
       rpy="-1.9723E-15 2.4325E-31 0" />
     <parent
-      link="komodo_$(arg komodo_id)_base_link" />
-    <child
-      link="komodo_$(arg komodo_id)_Asus_Camera_link" />
+      link="base_link" />
+    <child
+      link="Asus_Camera_link" />
     <axis
       xyz="0 0 0" />
   </joint>
   <link
-    name="komodo_$(arg komodo_id)_Arm_base_link">
+    name="Arm_base_link">
     <inertial>
       <origin
@@ -624,5 +624,5 @@
   </link>
   <joint
-    name="komodo_$(arg komodo_id)_Arm_base_joint"
+    name="Arm_base_joint"
     type="fixed">
     <origin
@@ -630,12 +630,12 @@
       rpy="1.5708 -1.9723E-15 -1.5708" />
     <parent
-      link="komodo_$(arg komodo_id)_base_link" />
-    <child
-      link="komodo_$(arg komodo_id)_Arm_base_link" />
+      link="base_link" />
+    <child
+      link="Arm_base_link" />
     <axis
       xyz="0 0 0" />
   </joint>
   <link
-    name="komodo_$(arg komodo_id)_base_rotation_link">
+    name="base_rotation_link">
     <inertial>
       <origin
@@ -677,5 +677,5 @@
   </link>
   <joint
-    name="komodo_$(arg komodo_id)_base_rotation_joint"
+    name="base_rotation_joint"
     type="revolute">
     <origin
@@ -683,7 +683,7 @@
       rpy="-1.5708 1.5708 0" />
     <parent
-      link="komodo_$(arg komodo_id)_Arm_base_link" />
-    <child
-      link="komodo_$(arg komodo_id)_base_rotation_link" />
+      link="Arm_base_link" />
+    <child
+      link="base_rotation_link" />
     <axis
       xyz="0 0 1" />
@@ -695,5 +695,5 @@
   </joint>
   <link
-    name="komodo_$(arg komodo_id)_shoulder_link">
+    name="shoulder_link">
     <inertial>
       <origin
@@ -735,5 +735,5 @@
   </link>
   <joint
-    name="komodo_$(arg komodo_id)_shoulder_joint"
+    name="shoulder_joint"
     type="revolute">
     <origin
@@ -741,7 +741,7 @@
       rpy="0 0 0" />
     <parent
-      link="komodo_$(arg komodo_id)_base_rotation_link" />
-    <child
-      link="komodo_$(arg komodo_id)_shoulder_link" />
+      link="base_rotation_link" />
+    <child
+      link="shoulder_link" />
     <axis
       xyz="0 1 0" />
@@ -753,5 +753,5 @@
   </joint>
   <link
-    name="komodo_$(arg komodo_id)_elbow1_link">
+    name="elbow1_link">
     <inertial>
       <origin
@@ -793,5 +793,5 @@
   </link>
   <joint
-    name="komodo_$(arg komodo_id)_elbow1_joint"
+    name="elbow1_joint"
     type="revolute">
     <origin
@@ -799,7 +799,7 @@
       rpy="0 0 0" />
     <parent
-      link="komodo_$(arg komodo_id)_shoulder_link" />
-    <child
-      link="komodo_$(arg komodo_id)_elbow1_link" />
+      link="shoulder_link" />
+    <child
+      link="elbow1_link" />
     <axis
       xyz="-1 0 0" />
@@ -811,5 +811,5 @@
   </joint>
   <link
-    name="komodo_$(arg komodo_id)_elbow2_link">
+    name="elbow2_link">
     <inertial>
       <origin
@@ -851,5 +851,5 @@
   </link>
   <joint
-    name="komodo_$(arg komodo_id)_elbow2_joint"
+    name="elbow2_joint"
     type="revolute">
     <origin
@@ -857,7 +857,7 @@
       rpy="0 1.7393E-18 0" />
     <parent
-      link="komodo_$(arg komodo_id)_elbow1_link" />
-    <child
-      link="komodo_$(arg komodo_id)_elbow2_link" />
+      link="elbow1_link" />
+    <child
+      link="elbow2_link" />
     <axis
       xyz="0 1 0" />
@@ -869,5 +869,5 @@
   </joint>
   <link
-    name="komodo_$(arg komodo_id)_wrist_link">
+    name="wrist_link">
     <inertial>
       <origin
@@ -909,5 +909,5 @@
   </link>
   <joint
-    name="komodo_$(arg komodo_id)_wrist_joint"
+    name="wrist_joint"
     type="revolute">
     <origin
@@ -915,7 +915,7 @@
       rpy="0 1.1023E-34 0" />
     <parent
-      link="komodo_$(arg komodo_id)_elbow2_link" />
-    <child
-      link="komodo_$(arg komodo_id)_wrist_link" />
+      link="elbow2_link" />
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