Commit message: fixes

File: ric_description/komodo/komodo.xacro (robot description, xacro)
@@ -1,150 +1,96 @@
 <?xml version="1.0"?>
 <robot xmlns:xacro="http://www.ros.org/wiki/ric" name="ric_description">
-<xacro:property name="komodo_color" value="0 0.517 0.26 1" />
   <link
     name="komodo_$(arg komodo_id)_base_link">
     <inertial>
       <origin
-        xyz="-0.036889 0.00027038 0.069426"
-        rpy="0 0 0" />
-      <mass
-        value="4.706" />
-      <inertia
-        ixx="0.032024"
-        ixy="0.00038846"
-        ixz="-0.0046108"
-        iyy="0.065583"
-        iyz="2.8552E-06"
-        izz="0.076391" />
-    </inertial>
-    <visual>
-      <origin
-        xyz="0 0 0"
-        rpy="0 0 0" />
-      <geometry>
-        <mesh
-          filename="package://ric_description/lizi/meshes/base_link.STL" />
-      </geometry>
-      <material
-        name="">
-        <color
-          rgba="${komodo_color}" />
-      </material>
-    </visual>
-    <collision>
-      <origin
-        xyz="0 0 0"
-        rpy="0 0 0" />
-      <geometry>
-        <mesh
-          filename="package://ric_description/lizi/meshes/base_link.STL" />
-      </geometry>
-    </collision>
-  </link>
-  <link
-    name="komodo_$(arg komodo_id)_FL_Wheel_link">
-    <inertial>
-      <origin
-        xyz="2.9411E-11 -0.0075967 5.8231E-11"
-        rpy="0 0 0" />
-      <mass
-        value="0.4084" />
-      <inertia
-        ixx="0.00059356"
-        ixy="3.4979E-14"
-        ixz="-4.6514E-14"
-        iyy="0.0011268"
-        iyz="5.6928E-14"
-        izz="0.00059356" />
-    </inertial>
-    <visual>
-      <origin
-        xyz="0 0 0"
-        rpy="0 0 0" />
-      <geometry>
-        <mesh
-          filename="package://ric_description/lizi/meshes/FL_Wheel_Link.STL" />
-      </geometry>
-      <material
-        name="">
-        <color
-          rgba="0.2 0.2 0.2 1" />
-      </material>
-    </visual>
-    <collision>
-      <origin
-        xyz="0 0 0"
-        rpy="0 0 0" />
-      <geometry>
-        <mesh
-          filename="package://ric_description/lizi/meshes/FL_Wheel_Link.STL" />
-      </geometry>
-    </collision>
-  </link>
-  <joint
-    name="komodo_$(arg komodo_id)_FL_Wheel_Joint"
-    type="continuous">
-    <origin
-      xyz="0.118 0.1338 0.026"
-      rpy="0 0 -1.3371E-16" />
+        xyz="-0.015958 -0.00012764 0.018284"
+        rpy="0 0 0" />
+      <mass
+        value="8.0792" />
+      <inertia
+        ixx="0.080966"
+        ixy="-0.00012771"
+        ixz="-0.016999"
+        iyy="0.17431"
+        iyz="6.1541E-05"
+        izz="0.23493" />
+    </inertial>
+    <visual>
+      <origin
+        xyz="0 0 0"
+        rpy="0 0 0" />
+      <geometry>
+        <mesh
+          filename="package://ric_description/komodo/meshes/base_link.STL" />
+      </geometry>
+      <material
+        name="">
+        <color
+          rgba="0.25294 0.25294 0.25294 1" />
+      </material>
+    </visual>
+    <collision>
+      <origin
+        xyz="0 0 0"
+        rpy="0 0 0" />
+      <geometry>
+        <mesh
+          filename="package://ric_description/komodo/meshes/base_link.STL" />
+      </geometry>
+    </collision>
+  </link>
+  <link
+    name="komodo_$(arg komodo_id)_FR_Wheel_link">
+    <inertial>
+      <origin
+        xyz="-6.3555E-05 5.4825E-06 4.0333E-11"
+        rpy="0 0 0" />
+      <mass
+        value="3.0437" />
+      <inertia
+        ixx="0.028387"
+        ixy="1.0601E-09"
+        ixz="3.2946E-12"
+        iyy="0.015485"
+        iyz="1.2761E-10"
+        izz="0.015484" />
+    </inertial>
+    <visual>
+      <origin
+        xyz="0 0 0"
+        rpy="0 0 0" />
+      <geometry>
+        <mesh
+          filename="package://ric_description/komodo/meshes/FR_Wheel_link.STL" />
+      </geometry>
+      <material
+        name="">
+        <color
+          rgba="0.45294 0.45294 0.45294 1" />
+      </material>
+    </visual>
+    <collision>
+      <origin
+        xyz="0 0 0"
+        rpy="0 0 0" />
+      <geometry>
+        <mesh
+          filename="package://ric_description/komodo/meshes/FR_Wheel_link.STL" />
+      </geometry>
+    </collision>
+  </link>
+  <joint
+    name="komodo_$(arg komodo_id)_FR_Wheel_joint"
+    type="fixed">
+    <origin
+      xyz="0.165 -0.18938 0"
+      rpy="-2.4325E-31 -1.9723E-15 -1.5708" />
     <parent
       link="komodo_$(arg komodo_id)_base_link" />
     <child
-      link="komodo_$(arg komodo_id)_FL_Wheel_link" />
-    <axis
-      xyz="0 -1 0" />
-  </joint>
-  <link
-    name="komodo_$(arg komodo_id)_RL_Wheel_link">
-    <inertial>
-      <origin
-        xyz="2.9411E-11 -0.0035967 5.8231E-11"
-        rpy="0 0 0" />
-      <mass
-        value="0.4084" />
-      <inertia
-        ixx="0.00059356"
-        ixy="3.4979E-14"
-        ixz="-4.6514E-14"
-        iyy="0.0011268"
-        iyz="5.6928E-14"
-        izz="0.00059356" />
-    </inertial>
-    <visual>
-      <origin
-        xyz="0 0 0"
-        rpy="0 0 0" />
-      <geometry>
-        <mesh
-          filename="package://ric_description/lizi/meshes/RL_Wheel_Link.STL" />
-      </geometry>
-      <material
-        name="">
-        <color
-          rgba="0.2 0.2 0.2 1" />
-      </material>
-    </visual>
-    <collision>
-      <origin
-        xyz="0 0 0"
-        rpy="0 0 0" />
-      <geometry>
-        <mesh
-          filename="package://ric_description/lizi/meshes/RL_Wheel_Link.STL" />
-      </geometry>
-    </collision>
-  </link>
-  <joint
-    name="komodo_$(arg komodo_id)_RL_Wheel_Joint"
-    type="continuous">
-    <origin
-      xyz="-0.118 0.1338 0.026"
-      rpy="0 0 -6.6853E-16" />
-    <parent
-      link="komodo_$(arg komodo_id)_base_link" />
-    <child
-      link="komodo_$(arg komodo_id)_RL_Wheel_link" />
-    <axis
-      xyz="0 -1 0" />
+      link="komodo_$(arg komodo_id)_FR_Wheel_link" />
+    <axis
+      xyz="-1 0 0" />
     <limit
       effort="0"
@@ -152,161 +98,55 @@
   </joint>
   <link
-    name="komodo_$(arg komodo_id)_RR_Wheel_link">
-    <inertial>
-      <origin
-        xyz="-2.9411E-11 0.0035967 5.8231E-11"
-        rpy="0 0 0" />
-      <mass
-        value="0.4084" />
-      <inertia
-        ixx="0.00059356"
-        ixy="3.4979E-14"
-        ixz="4.6514E-14"
-        iyy="0.0011268"
-        iyz="-5.6928E-14"
-        izz="0.00059356" />
-    </inertial>
-    <visual>
-      <origin
-        xyz="0 0 0"
-        rpy="0 0 0" />
-      <geometry>
-        <mesh
-          filename="package://ric_description/lizi/meshes/RR_Wheel_Link.STL" />
-      </geometry>
-      <material
-        name="">
-        <color
-          rgba="0.2 0.2 0.2 1" />
-      </material>
-    </visual>
-    <collision>
-      <origin
-        xyz="0 0 0"
-        rpy="0 0 0" />
-      <geometry>
-        <mesh
-          filename="package://ric_description/lizi/meshes/RR_Wheel_Link.STL" />
-      </geometry>
-    </collision>
-  </link>
-  <joint
-    name="komodo_$(arg komodo_id)_RR_Wheel_Joint"
-    type="continuous">
-    <origin
-      xyz="-0.118 -0.1338 0.026"
-      rpy="-1.2938E-16 -1.2938E-15 -6.6853E-16" />
+    name="komodo_$(arg komodo_id)_FL_Wheel_link">
+    <inertial>
+      <origin
+        xyz="-6.3555E-05 1.6687E-11 5.4825E-06"
+        rpy="0 0 0" />
+      <mass
+        value="3.0437" />
+      <inertia
+        ixx="0.028387"
+        ixy="-9.3612E-13"
+        ixz="1.0621E-09"
+        iyy="0.015484"
+        iyz="-1.2165E-10"
+        izz="0.015485" />
+    </inertial>
+    <visual>
+      <origin
+        xyz="0 0 0"
+        rpy="0 0 0" />
+      <geometry>
+        <mesh
+          filename="package://ric_description/komodo/meshes/FL_Wheel_link.STL" />
+      </geometry>
+      <material
+        name="">
+        <color
+          rgba="0.45294 0.45294 0.45294 1" />
+      </material>
+    </visual>
+    <collision>
+      <origin
+        xyz="0 0 0"
+        rpy="0 0 0" />
+      <geometry>
+        <mesh
+          filename="package://ric_description/komodo/meshes/FL_Wheel_link.STL" />
+      </geometry>
+    </collision>
+  </link>
+  <joint
+    name="komodo_$(arg komodo_id)_FL_Wheel_joint"
+    type="fixed">
+    <origin
+      xyz="0.165 0.18938 0"
+      rpy="2.4325E-31 1.9723E-15 1.5708" />
     <parent
       link="komodo_$(arg komodo_id)_base_link" />
     <child
-      link="komodo_$(arg komodo_id)_RR_Wheel_link" />
-    <axis
-      xyz="0 1 0" />
-  </joint>
-  <link
-    name="komodo_$(arg komodo_id)_FR_Wheel_link">
-    <inertial>
-      <origin
-        xyz="-2.9052E-11 0.0035967 5.8411E-11"
-        rpy="0 0 0" />
-      <mass
-        value="0.4084" />
-      <inertia
-        ixx="0.00059356"
-        ixy="3.4627E-14"
-        ixz="4.9977E-14"
-        iyy="0.0011268"
-        iyz="-5.7142E-14"
-        izz="0.00059356" />
-    </inertial>
-    <visual>
-      <origin
-        xyz="0 0 0"
-        rpy="0 0 0" />
-      <geometry>
-        <mesh
-          filename="package://ric_description/lizi/meshes/FR_Wheel_Link.STL" />
-      </geometry>
-      <material
-        name="">
-        <color
-          rgba="0.2 0.2 0.2 1" />
-      </material>
-    </visual>
-    <collision>
-      <origin
-        xyz="0 0 0"
-        rpy="0 0 0" />
-      <geometry>
-        <mesh
-          filename="package://ric_description/lizi/meshes/FR_Wheel_Link.STL" />
-      </geometry>
-    </collision>
-  </link>
-  <joint
-    name="komodo_$(arg komodo_id)_FR_Wheel_Joint"
-    type="continuous">
-    <origin
-      xyz="0.118 -0.1338 0.026"
-      rpy="4.4216E-16 -0.0061583 -2.6824E-16" />
-    <parent
-      link="komodo_$(arg komodo_id)_base_link" />
-    <child
-      link="komodo_$(arg komodo_id)_FR_Wheel_link" />
-    <axis
-      xyz="0 1 0" />
-  </joint>
-  <link
-    name="komodo_$(arg komodo_id)_Asus_Pan_link">
-    <inertial>
-      <origin
-        xyz="-0.015533 -0.010751 0.019512"
-        rpy="0 0 0" />
-      <mass
-        value="0.016162" />
-      <inertia
-        ixx="5.2781E-06"
-        ixy="1.178E-06"
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
Commit message: fixes

File: ric_description/komodo/komodo.xacro (robot description, xacro)
@@ -425,5 +425,5 @@
   </joint>
   <link
-    name="komodo_$(arg komodo_id)_Front_Camera_optical_link">
+    name="komodo_$(arg komodo_id)_Front_Camera_link">
     <inertial>
       <origin
@@ -446,5 +446,5 @@
       <geometry>
         <mesh
-          filename="package://ric_description/komodo/meshes/Front_Camera_optical_link.STL" />
+          filename="package://ric_description/komodo/meshes/Front_Camera_link.STL" />
       </geometry>
       <material
@@ -460,10 +460,10 @@
       <geometry>
         <mesh
-          filename="package://ric_description/komodo/meshes/Front_Camera_optical_link.STL" />
-      </geometry>
-    </collision>
-  </link>
-  <joint
-    name="komodo_$(arg komodo_id)_Front_Camera_optical_joint"
+          filename="package://ric_description/komodo/meshes/Front_Camera_link.STL" />
+      </geometry>
+    </collision>
+  </link>
+  <joint
+    name="komodo_$(arg komodo_id)_Front_Camera_joint"
     type="fixed">
     <origin
@@ -473,5 +473,5 @@
       link="komodo_$(arg komodo_id)_base_link" />
     <child
-      link="komodo_$(arg komodo_id)_Front_Camera_optical_link" />
+      link="komodo_$(arg komodo_id)_Front_Camera_link" />
     <axis
       xyz="0 0 0" />
@@ -531,5 +531,5 @@
   </joint>
   <link
-    name="komodo_$(arg komodo_id)_Asus_link">
+    name="komodo_$(arg komodo_id)_Asus_Camera_link">
     <inertial>
       <origin
@@ -552,5 +552,5 @@
       <geometry>
         <mesh
-          filename="package://ric_description/komodo/meshes/Asus_link.STL" />
+          filename="package://ric_description/komodo/meshes/Asus_Camera_link.STL" />
       </geometry>
       <material
@@ -566,5 +566,5 @@
       <geometry>
         <mesh
-          filename="package://ric_description/komodo/meshes/Asus_link.STL" />
+          filename="package://ric_description/komodo/meshes/Asus_Camera_link.STL" />
       </geometry>
     </collision>
@@ -579,5 +579,5 @@
       link="komodo_$(arg komodo_id)_base_link" />
     <child
-      link="komodo_$(arg komodo_id)_Asus_link" />
+      link="komodo_$(arg komodo_id)_Asus_Camera_link" />
     <axis
       xyz="0 0 0" />
@@ -1043,5 +1043,5 @@
   </joint>
   <link
-    name="komodo_$(arg komodo_id)_Arm_camera_link">
+    name="komodo_$(arg komodo_id)_Arm_Camera_link">
     <inertial>
       <origin
@@ -1064,5 +1064,5 @@
       <geometry>
         <mesh
-          filename="package://ric_description/komodo/meshes/Arm_camera_link.STL" />
+          filename="package://ric_description/komodo/meshes/Arm_Camera_link.STL" />
       </geometry>
       <material
@@ -1078,5 +1078,5 @@
       <geometry>
         <mesh
-          filename="package://ric_description/komodo/meshes/Arm_camera_link.STL" />
+          filename="package://ric_description/komodo/meshes/Arm_Camera_link.STL" />
       </geometry>
     </collision>
@@ -1091,5 +1091,5 @@
       link="komodo_$(arg komodo_id)_wrist_link" />
     <child
-      link="komodo_$(arg komodo_id)_Arm_camera_link" />
+      link="komodo_$(arg komodo_id)_Arm_Camera_link" />
     <axis
       xyz="0 0 0" />
