Commit message: fixes

File: ric_description/komodo/komodo.xacro (robot description, xacro)
@@ -23,19 +23,19 @@
       <geometry>
         <mesh
-          filename="package://komodo_urdf/meshes/base_link.STL" />
-      </geometry>
-      <material
-        name="">
-        <color
-          rgba="0.752941176470588 0.752941176470588 0.752941176470588 1" />
-      </material>
-    </visual>
-    <collision>
-      <origin
-        xyz="0 0 0"
-        rpy="0 0 0" />
-      <geometry>
-        <mesh
-          filename="package://komodo_urdf/meshes/base_link.STL" />
+          filename="package://ric_description/komodo/meshes/base_link.STL" />
+      </geometry>
+      <material
+        name="">
+        <color
+          rgba="0.752941176470588 0.752941176470588 0.752941176470588 1" />
+      </material>
+    </visual>
+    <collision>
+      <origin
+        xyz="0 0 0"
+        rpy="0 0 0" />
+      <geometry>
+        <mesh
+          filename="package://ric_description/komodo/meshes/base_link.STL" />
       </geometry>
     </collision>
@@ -63,19 +63,19 @@
       <geometry>
         <mesh
-          filename="package://komodo_urdf/meshes/FR_Wheel_link.STL" />
-      </geometry>
-      <material
-        name="">
-        <color
-          rgba="0.752941176470588 0.752941176470588 0.752941176470588 1" />
-      </material>
-    </visual>
-    <collision>
-      <origin
-        xyz="0 0 0"
-        rpy="0 0 0" />
-      <geometry>
-        <mesh
-          filename="package://komodo_urdf/meshes/FR_Wheel_link.STL" />
+          filename="package://ric_description/komodo/meshes/FR_Wheel_link.STL" />
+      </geometry>
+      <material
+        name="">
+        <color
+          rgba="0.752941176470588 0.752941176470588 0.752941176470588 1" />
+      </material>
+    </visual>
+    <collision>
+      <origin
+        xyz="0 0 0"
+        rpy="0 0 0" />
+      <geometry>
+        <mesh
+          filename="package://ric_description/komodo/meshes/FR_Wheel_link.STL" />
       </geometry>
     </collision>
@@ -116,19 +116,19 @@
       <geometry>
         <mesh
-          filename="package://komodo_urdf/meshes/FL_Wheel_link.STL" />
-      </geometry>
-      <material
-        name="">
-        <color
-          rgba="0.752941176470588 0.752941176470588 0.752941176470588 1" />
-      </material>
-    </visual>
-    <collision>
-      <origin
-        xyz="0 0 0"
-        rpy="0 0 0" />
-      <geometry>
-        <mesh
-          filename="package://komodo_urdf/meshes/FL_Wheel_link.STL" />
+          filename="package://ric_description/komodo/meshes/FL_Wheel_link.STL" />
+      </geometry>
+      <material
+        name="">
+        <color
+          rgba="0.752941176470588 0.752941176470588 0.752941176470588 1" />
+      </material>
+    </visual>
+    <collision>
+      <origin
+        xyz="0 0 0"
+        rpy="0 0 0" />
+      <geometry>
+        <mesh
+          filename="package://ric_description/komodo/meshes/FL_Wheel_link.STL" />
       </geometry>
     </collision>
@@ -169,19 +169,19 @@
       <geometry>
         <mesh
-          filename="package://komodo_urdf/meshes/RR_Wheel_link.STL" />
-      </geometry>
-      <material
-        name="">
-        <color
-          rgba="0.752941176470588 0.752941176470588 0.752941176470588 1" />
-      </material>
-    </visual>
-    <collision>
-      <origin
-        xyz="0 0 0"
-        rpy="0 0 0" />
-      <geometry>
-        <mesh
-          filename="package://komodo_urdf/meshes/RR_Wheel_link.STL" />
+          filename="package://ric_description/komodo/meshes/RR_Wheel_link.STL" />
+      </geometry>
+      <material
+        name="">
+        <color
+          rgba="0.752941176470588 0.752941176470588 0.752941176470588 1" />
+      </material>
+    </visual>
+    <collision>
+      <origin
+        xyz="0 0 0"
+        rpy="0 0 0" />
+      <geometry>
+        <mesh
+          filename="package://ric_description/komodo/meshes/RR_Wheel_link.STL" />
       </geometry>
     </collision>
@@ -222,19 +222,19 @@
       <geometry>
         <mesh
-          filename="package://komodo_urdf/meshes/RL_Wheel_link.STL" />
-      </geometry>
-      <material
-        name="">
-        <color
-          rgba="0.752941176470588 0.752941176470588 0.752941176470588 1" />
-      </material>
-    </visual>
-    <collision>
-      <origin
-        xyz="0 0 0"
-        rpy="0 0 0" />
-      <geometry>
-        <mesh
-          filename="package://komodo_urdf/meshes/RL_Wheel_link.STL" />
+          filename="package://ric_description/komodo/meshes/RL_Wheel_link.STL" />
+      </geometry>
+      <material
+        name="">
+        <color
+          rgba="0.752941176470588 0.752941176470588 0.752941176470588 1" />
+      </material>
+    </visual>
+    <collision>
+      <origin
+        xyz="0 0 0"
+        rpy="0 0 0" />
+      <geometry>
+        <mesh
+          filename="package://ric_description/komodo/meshes/RL_Wheel_link.STL" />
       </geometry>
     </collision>
@@ -275,19 +275,19 @@
       <geometry>
         <mesh
-          filename="package://komodo_urdf/meshes/Left_URF_link.STL" />
-      </geometry>
-      <material
-        name="">
-        <color
-          rgba="0.752941176470588 0.752941176470588 0.752941176470588 1" />
-      </material>
-    </visual>
-    <collision>
-      <origin
-        xyz="0 0 0"
-        rpy="0 0 0" />
-      <geometry>
-        <mesh
-          filename="package://komodo_urdf/meshes/Left_URF_link.STL" />
+          filename="package://ric_description/komodo/meshes/Left_URF_link.STL" />
+      </geometry>
+      <material
+        name="">
+        <color
+          rgba="0.752941176470588 0.752941176470588 0.752941176470588 1" />
+      </material>
+    </visual>
+    <collision>
+      <origin
+        xyz="0 0 0"
+        rpy="0 0 0" />
+      <geometry>
+        <mesh
+          filename="package://ric_description/komodo/meshes/Left_URF_link.STL" />
       </geometry>
     </collision>
@@ -328,19 +328,19 @@
       <geometry>
         <mesh
-          filename="package://komodo_urdf/meshes/Rear_URF_link.STL" />
-      </geometry>
-      <material
-        name="">
-        <color
-          rgba="0.752941176470588 0.752941176470588 0.752941176470588 1" />
-      </material>
-    </visual>
-    <collision>
-      <origin
-        xyz="0 0 0"
-        rpy="0 0 0" />
-      <geometry>
-        <mesh
-          filename="package://komodo_urdf/meshes/Rear_URF_link.STL" />
+          filename="package://ric_description/komodo/meshes/Rear_URF_link.STL" />
+      </geometry>
+      <material
+        name="">
+        <color
+          rgba="0.752941176470588 0.752941176470588 0.752941176470588 1" />
+      </material>
+    </visual>
+    <collision>
+      <origin
+        xyz="0 0 0"
+        rpy="0 0 0" />
+      <geometry>
+        <mesh
+          filename="package://ric_description/komodo/meshes/Rear_URF_link.STL" />
       </geometry>
     </collision>
@@ -381,19 +381,19 @@
       <geometry>
         <mesh
-          filename="package://komodo_urdf/meshes/Right_URF_link.STL" />
-      </geometry>
-      <material
-        name="">
-        <color
-          rgba="0.752941176470588 0.752941176470588 0.752941176470588 1" />
-      </material>
-    </visual>
-    <collision>
-      <origin
-        xyz="0 0 0"
-        rpy="0 0 0" />
-      <geometry>
-        <mesh
-          filename="package://komodo_urdf/meshes/Right_URF_link.STL" />
+          filename="package://ric_description/komodo/meshes/Right_URF_link.STL" />
+      </geometry>
+      <material
+        name="">
+        <color
+          rgba="0.752941176470588 0.752941176470588 0.752941176470588 1" />
+      </material>
+    </visual>
+    <collision>
+      <origin
+        xyz="0 0 0"
+        rpy="0 0 0" />
+      <geometry>
+        <mesh
+          filename="package://ric_description/komodo/meshes/Right_URF_link.STL" />
       </geometry>
     </collision>
@@ -434,5 +434,5 @@
       <geometry>
         <mesh
-          filename="package://komodo_urdf/meshes/Front_Camera_link.STL" />
+          filename="package://ric_description/komodo/meshes/Front_Camera_link.STL" />
       </geometry>
       <material
@@ -448,5 +448,5 @@
       <geometry>
         <mesh
-          filename="package://komodo_urdf/meshes/Front_Camera_link.STL" />
+          filename="package://ric_description/komodo/meshes/Front_Camera_link.STL" />
       </geometry>
     </collision>
@@ -487,5 +487,5 @@
       <geometry>
         <mesh
-          filename="package://komodo_urdf/meshes/Laser_link.STL" />
+          filename="package://ric_description/komodo/meshes/Laser_link.STL" />
       </geometry>
       <material
@@ -501,5 +501,5 @@
       <geometry>
         <mesh
-          filename="package://komodo_urdf/meshes/Laser_link.STL" />
+          filename="package://ric_description/komodo/meshes/Laser_link.STL" />
       </geometry>
     </collision>
@@ -540,5 +540,5 @@
       <geometry>
         <mesh
-          filename="package://komodo_urdf/meshes/Asus_Camera_link.STL" />
+          filename="package://ric_description/komodo/meshes/Asus_Camera_link.STL" />
       </geometry>
       <material
@@ -554,5 +554,5 @@
       <geometry>
         <mesh
-          filename="package://komodo_urdf/meshes/Asus_Camera_link.STL" />
+          filename="package://ric_description/komodo/meshes/Asus_Camera_link.STL" />
       </geometry>
     </collision>
@@ -593,19 +593,19 @@
       <geometry>
         <mesh
-          filename="package://komodo_urdf/meshes/Arm_base_link.STL" />
-      </geometry>
-      <material
-        name="">
-        <color
-          rgba="0.752941176470588 0.752941176470588 0.752941176470588 1" />
-      </material>
-    </visual>
-    <collision>
-      <origin
-        xyz="0 0 0"
-        rpy="0 0 0" />
-      <geometry>
-        <mesh
-          filename="package://komodo_urdf/meshes/Arm_base_link.STL" />
+          filename="package://ric_description/komodo/meshes/Arm_base_link.STL" />
+      </geometry>
+      <material
+        name="">
+        <color
+          rgba="0.752941176470588 0.752941176470588 0.752941176470588 1" />
+      </material>
+    </visual>
+    <collision>
+      <origin
+        xyz="0 0 0"
+        rpy="0 0 0" />
+      <geometry>
+        <mesh
+          filename="package://ric_description/komodo/meshes/Arm_base_link.STL" />
       </geometry>
     </collision>
@@ -646,19 +646,19 @@
       <geometry>
         <mesh
-          filename="package://komodo_urdf/meshes/base_rotation_link.STL" />
-      </geometry>
-      <material
-        name="">
-        <color
-          rgba="0.752941176470588 0.752941176470588 0.752941176470588 1" />
-      </material>
-    </visual>
-    <collision>
-      <origin
-        xyz="0 0 0"
-        rpy="0 0 0" />
-      <geometry>
-        <mesh
-          filename="package://komodo_urdf/meshes/base_rotation_link.STL" />
+          filename="package://ric_description/komodo/meshes/base_rotation_link.STL" />
+      </geometry>
+      <material
+        name="">
+        <color
+          rgba="0.752941176470588 0.752941176470588 0.752941176470588 1" />
+      </material>
+    </visual>
+    <collision>
+      <origin
+        xyz="0 0 0"
+        rpy="0 0 0" />
+      <geometry>
+        <mesh
+          filename="package://ric_description/komodo/meshes/base_rotation_link.STL" />
       </geometry>
     </collision>
@@ -704,19 +704,19 @@
       <geometry>
         <mesh
-          filename="package://komodo_urdf/meshes/shoulder_link.STL" />
-      </geometry>
-      <material
-        name="">
-        <color
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