Commit message: added komodo gazobo simulation

File: ric_description/komodo/komodo.xacro (robot description, xacro)
@@ -8,12 +8,12 @@
         rpy="0 0 0" />
       <mass
-        value="4.50894999160313" />
-      <inertia
-        ixx="0.0723503030508731"
-        ixy="-4.68485359152423E-05"
-        ixz="-0.00875564429068847"
-        iyy="0.138127064231828"
-        iyz="1.19695110167269E-05"
-        izz="0.194371448739423" />
+        value="45.0894999160313" />
+      <inertia
+        ixx="0.723503030508731"
+        ixy="-46.8485359152423E-05"
+        ixz="-0.0875564429068847"
+        iyy="1.38127064231828"
+        iyz="11.9695110167269E-05"
+        izz="1.94371448739423" />
     </inertial>
     <visual>
@@ -33,5 +33,5 @@
     <collision>
       <origin
-        xyz="0 0 0"
+        xyz="-0.065 0 0"
         rpy="0 0 0" />
       <geometry>
@@ -74,8 +74,10 @@
       <origin
         xyz="0 0 0"
-        rpy="0 0 0" />
-      <geometry>
-        <mesh
-          filename="package://ric_description/komodo/meshes/FR_Wheel_link.STL" />
+        rpy="0 1.5 0" />
+      <geometry>
+       <!--mesh
+          filename="package://ric_description/komodo/meshes_elevator/FR_Wheel_link.STL" /-->
+        <cylinder length="0.05" radius="0.1"
+          />
       </geometry>
     </collision>
@@ -86,5 +88,5 @@
     <origin
       xyz="0.173999999999995 -0.2009 0"
-      rpy="2.62229105359916E-15 6.9308460464278E-17 -1.5707963267949" />
+      rpy="2.62229105359916E-15 6.9308460464278E-17 1.5707963267949" />
     <parent
       link="komodo_$(arg komodo_id)_base_link" />
@@ -127,8 +129,10 @@
       <origin
         xyz="0 0 0"
-        rpy="0 0 0" />
-      <geometry>
-        <mesh
-          filename="package://ric_description/komodo/meshes/FL_Wheel_link.STL" />
+        rpy="0 1.5 0" />
+      <geometry>
+       <!--mesh
+          filename="package://ric_description/komodo/meshes_elevator/FR_Wheel_link.STL" /-->
+        <cylinder length="0.05" radius="0.1"
+          />
       </geometry>
     </collision>
@@ -139,5 +143,5 @@
     <origin
       xyz="0.173999999999995 0.2009 0"
-      rpy="-2.62229105359916E-15 6.93084604642783E-17 1.5707963267949" />
+      rpy="-2.62229105359916E-15 6.93084604642783E-17 -1.5707963267949" />
     <parent
       link="komodo_$(arg komodo_id)_base_link" />
@@ -180,8 +184,10 @@
       <origin
         xyz="0 0 0"
-        rpy="0 0 0" />
-      <geometry>
-        <mesh
-          filename="package://ric_description/komodo/meshes/RR_Wheel_link.STL" />
+        rpy="0 1.5 0" />
+      <geometry>
+       <!--mesh
+          filename="package://ric_description/komodo/meshes_elevator/FR_Wheel_link.STL" /-->
+        <cylinder length="0.05" radius="0.1"
+          />
       </geometry>
     </collision>
@@ -192,5 +198,5 @@
     <origin
       xyz="-0.156000000000005 -0.2009 0"
-      rpy="2.62229105359916E-15 -1.59433090848306E-31 -1.5707963267949" />
+      rpy="2.62229105359916E-15 -1.59433090848306E-31 1.5707963267949" />
     <parent
       link="komodo_$(arg komodo_id)_base_link" />
@@ -233,8 +239,10 @@
       <origin
         xyz="0 0 0"
-        rpy="0 0 0" />
-      <geometry>
-        <mesh
-          filename="package://ric_description/komodo/meshes/RL_Wheel_link.STL" />
+        rpy="0 1.5 0" />
+      <geometry>
+       <!--mesh
+          filename="package://ric_description/komodo/meshes_elevator/FR_Wheel_link.STL" /-->
+        <cylinder length="0.05" radius="0.1"
+          />
       </geometry>
     </collision>
@@ -245,5 +253,5 @@
     <origin
       xyz="-0.156000000000005 0.2009 0"
-      rpy="-2.62229105359916E-15 -5.57680208627196E-32 1.5707963267949" />
+      rpy="-2.62229105359916E-15 -5.57680208627196E-32 -1.5707963267949" />
     <parent
       link="komodo_$(arg komodo_id)_base_link" />
@@ -280,5 +288,5 @@
         name="">
         <color
-          rgba="0.1 0.1 0.1 1" />
+          rgba="0.752941176470588 0.752941176470588 0.752941176470588 1" />
       </material>
     </visual>
@@ -333,5 +341,5 @@
         name="">
         <color
-          rgba="0.1 0.1 0.1 1" />
+          rgba="0.752941176470588 0.752941176470588 0.752941176470588 1" />
       </material>
     </visual>
@@ -386,5 +394,5 @@
         name="">
         <color
-          rgba="0.1 0.1 0.1 1" />
+          rgba="0.752941176470588 0.752941176470588 0.752941176470588 1" />
       </material>
     </visual>
@@ -677,7 +685,7 @@
       xyz="0 0 1" />
     <limit
-      lower="-1.57079"
-      upper="1.57079"
-      effort="0"
+      lower="-3.14"
+      upper="3.14"
+      effort="10"
       velocity="0" />
   </joint>
@@ -735,7 +743,7 @@
       xyz="0 1 0" />
     <limit
-      lower="-1.692969"
-      upper="1.692969"
-      effort="0"
+      lower="-1.57"
+      upper="1.57"
+      effort="2000"
       velocity="0" />
   </joint>
@@ -793,7 +801,7 @@
       xyz="-0.999999999998754 0 0" />
     <limit
-      lower="-2.4434"
-      upper="2.4434"
-      effort="0"
+      lower="-3.14"
+      upper="3.14"
+      effort="100"
       velocity="0" />
   </joint>
@@ -807,5 +815,5 @@
         value="1.12138857800426" />
       <inertia
-        ixx="0.0110599202589784"
+        ixx="0.0011156254663426"
         ixy="3.04261287700186E-07"
         ixz="-1.22468079415109E-06"
@@ -843,5 +851,5 @@
     <origin
       xyz="0 0 0.223999999999899"
-      rpy="-4.51048856041191E-16 3.35869632765754E-16 1.57079632687657" />
+      rpy="-4.51048856041191E-16 3.35869632765754E-16 0" />
     <parent
       link="komodo_$(arg komodo_id)_elbow1_link" />
@@ -849,9 +857,9 @@
       link="komodo_$(arg komodo_id)_elbow2_link" />
     <axis
-      xyz="1 0 0" />
+      xyz="0 1 0" />
     <limit
-      lower="-2.4434"
-      upper="2.4434"
-      effort="0"
+      lower="-3.14"
+      upper="3.14"
+      effort="10"
       velocity="0" />
   </joint>
@@ -860,5 +868,5 @@
     <inertial>
       <origin
-        xyz="-0.000140374211043626 4.00707618562063E-10 0.0303673809619358"
+        xyz="0 0 0"
         rpy="0 0 0" />
       <mass
@@ -883,5 +891,5 @@
         name="">
         <color
-          rgba="0.3 0.3 0.3 1" />
+          rgba="0.4 0.4 0.4 1" />
       </material>
     </visual>
@@ -900,6 +908,6 @@
     type="revolute">
     <origin
-      xyz="0 -0.0130999999999997 0.244749999999997"
-      rpy="-4.43972025628984E-16 -3.35842401421639E-15 -1.57079632687657" />
+      xyz="0.0137 0 0.244749999999997"
+      rpy="0 0 0" />
     <parent
       link="komodo_$(arg komodo_id)_elbow2_link" />
@@ -909,7 +917,7 @@
       xyz="0 0 0.999999999998754" />
     <limit
-      lower="-1.91986"
-      upper="1.91986"
-      effort="0"
+      lower="-3.14"
+      upper="3.14"
+      effort="10"
       velocity="0" />
   </joint>
@@ -923,15 +931,15 @@
         value="0.0111981711598485" />
       <inertia
-        ixx="9.77349829713274E-06"
-        ixy="6.1354405537333E-20"
-        ixz="3.95573177730842E-20"
-        iyy="1.11277552627936E-05"
-        iyz="2.19026618569787E-06"
-        izz="3.8860219521149E-06" />
-    </inertial>
-    <visual>
-      <origin
-        xyz="0 0 0"
-        rpy="0.185 0 0" />
+        ixx="0.000486392340366094"
+        ixy="4.20757000035677E-12"
+        ixz="-3.91843889020299E-06"
+        iyy="0.000211170064630335"
+        iyz="2.79335159568522E-12"
+        izz="0.000437528795624211" />
+    </inertial>
+    <visual>
+      <origin
+        xyz="0 0 0"
+        rpy="0 0 0" />
       <geometry>
         <mesh
@@ -967,7 +975,7 @@
       xyz="1 0 0" />
     <limit
-      lower="-0.87266"
-      upper="0.87266"
-      effort="0"
+      lower="-3.14"
+      upper="3.14"
+      effort="10"
       velocity="0" />
   </joint>
@@ -981,15 +989,15 @@
         value="0.0111981711598485" />
       <inertia
-        ixx="9.7734982971327E-06"
-        ixy="1.80407068651258E-20"
-        ixz="2.78908224261042E-20"
-        iyy="1.11277552627935E-05"
-        iyz="-2.19026618569788E-06"
-        izz="3.88602195211489E-06" />
-    </inertial>
-    <visual>
-      <origin
-        xyz="0 0 0"
-        rpy="-0.185 0 0" />
+        ixx="0.000486392340366094"
+        ixy="4.20757000035677E-12"
+        ixz="-3.91843889020299E-06"
+        iyy="0.000211170064630335"
+        iyz="2.79335159568522E-12"
+        izz="0.000437528795624211" />
+    </inertial>
+    <visual>
+      <origin
+        xyz="0 0 0"
+        rpy="0 0 0" />
       <geometry>
         <mesh
@@ -1025,7 +1033,7 @@
       xyz="1 0 0" />
     <limit
-      lower="-0.87266"
-      upper="0.87266"
-      effort="0"
+      lower="-3.14"
+      upper="3.14"
+      effort="10"
       velocity="0" />
   </joint>
@@ -1049,5 +1057,5 @@
       <origin
         xyz="0 0 0"
-        rpy="0 0 0" />
+        rpy="0 1.57 0" />
       <geometry>
         <mesh
@@ -1057,5 +1065,5 @@
         name="">
         <color
-          rgba="0.2 0.2 0.2 1" />
+          rgba="0.4 0.4 0.4 1" />
       </material>
     </visual>
@@ -1075,5 +1083,5 @@
     <origin
       xyz="-0.0552499999999999 0 0.0340250000000002"
-      rpy="1.60129334747211E-25 2.01127359533543E-16 -1.57079632649567" />
+      rpy="0 -1.57079632649567 0" />
     <parent
       link="komodo_$(arg komodo_id)_wrist_link" />
@@ -1136,3 +1144,474 @@
       xyz="1 0 0" />
   </joint>
+   <!-- ros_control plugin -->
+<gazebo>
+<plugin name="gazebo_ros_control" filename="libgazebo_ros_control.so">
+<robotNamespace>/komodo_$(arg komodo_id)</robotNamespace>
+</plugin>
+</gazebo>
+ <!-- Transmissions for ROS Control -->
+  <transmission name="tran1">
+    <type>transmission_interface/SimpleTransmission</type>
+    <joint name="komodo_$(arg komodo_id)_FR_Wheel_joint">
+<hardwareInterface>EffortJointInterface</hardwareInterface>
+    </joint>
+    <actuator name="motor1">
+      <hardwareInterface>EffortJointInterface</hardwareInterface>
+      <mechanicalReduction>1</mechanicalReduction>
+    </actuator>
+  </transmission>
+  <transmission name="tran2">
+    <type>transmission_interface/SimpleTransmission</type>
+    <joint name="komodo_$(arg komodo_id)_FL_Wheel_joint">
+<hardwareInterface>EffortJointInterface</hardwareInterface>
+    </joint>
+    <actuator name="motor2">
+      <hardwareInterface>EffortJointInterface</hardwareInterface>
+      <mechanicalReduction>1</mechanicalReduction>
+    </actuator>
+  </transmission>
+  <transmission name="tran3">
+    <type>transmission_interface/SimpleTransmission</type>
+    <joint name="komodo_$(arg komodo_id)_RR_Wheel_joint">
+<hardwareInterface>EffortJointInterface</hardwareInterface>
+    </joint>
+    <actuator name="motor3">
+      <hardwareInterface>EffortJointInterface</hardwareInterface>
+      <mechanicalReduction>1</mechanicalReduction>
+    </actuator>
+  </transmission>
+  <transmission name="tran4">
+    <type>transmission_interface/SimpleTransmission</type>
+    <joint name="komodo_$(arg komodo_id)_RL_Wheel_joint">
+<hardwareInterface>EffortJointInterface</hardwareInterface>
+    </joint>
+    <actuator name="motor4">
+      <hardwareInterface>EffortJointInterface</hardwareInterface>
+      <mechanicalReduction>1</mechanicalReduction>
+    </actuator>
+  </transmission>
+  <transmission name="tran5">
+    <type>transmission_interface/SimpleTransmission</type>
+    <joint name="komodo_$(arg komodo_id)_base_rotation_joint">
+<hardwareInterface>EffortJointInterface</hardwareInterface>
+    </joint>
+    <actuator name="motor5">
+      <hardwareInterface>EffortJointInterface</hardwareInterface>
+      <mechanicalReduction>1</mechanicalReduction>
+    </actuator>
+  </transmission>
+  <transmission name="tran6">
+    <type>transmission_interface/SimpleTransmission</type>
+    <joint name="komodo_$(arg komodo_id)_shoulder_joint">
+<hardwareInterface>EffortJointInterface</hardwareInterface>
+	</joint>
+    <actuator name="motor6">
+      <hardwareInterface>EffortJointInterface</hardwareInterface>
+      <mechanicalReduction>1</mechanicalReduction>
+    </actuator>
+  </transmission>
+  <transmission name="tran7">
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
Commit message: a

File: ric_description/komodo/komodo.xacro (robot description, xacro)
@@ -1,6 +1,25 @@
 <?xml version="1.0"?>
-<robot xmlns:xacro="http://www.ros.org/wiki/ric" name="ric_description">
-  <link
-    name="komodo_$(arg komodo_id)_base_link">
+<robot
+  name="komodo_$(arg komodo_id)">
+<!-- Dummy inertia link & Joint -->
+  <link
+    name="komodo_dummy_link">
+</link>
+  <joint
+    name="komodo_dummy_joint"
+    type="fixed">
+    <origin
+      xyz="0.0 0.0 0.0"
+      rpy="0 0 0" />
+    <parent
+      link="komodo_dummy_link" />
+    <child
+      link="komodo_base_link" />
+    <axis
+      xyz="0 0 0" />
+  </joint>
+<!-- Dummy link & node -->
+  <link
+    name="komodo_base_link">
     <inertial>
       <origin
@@ -42,5 +61,5 @@
   </link>
   <link
-    name="komodo_$(arg komodo_id)_FR_Wheel_link">
+    name="komodo_FR_Wheel_link">
     <inertial>
       <origin
@@ -84,5 +103,5 @@
   </link>
   <joint
-    name="komodo_$(arg komodo_id)_FR_Wheel_joint"
+    name="komodo_FR_Wheel_joint"
     type="continuous">
     <origin
@@ -90,12 +109,12 @@
       rpy="2.62229105359916E-15 6.9308460464278E-17 1.5707963267949" />
     <parent
-      link="komodo_$(arg komodo_id)_base_link" />
-    <child
-      link="komodo_$(arg komodo_id)_FR_Wheel_link" />
+      link="komodo_base_link" />
+    <child
+      link="komodo_FR_Wheel_link" />
     <axis
       xyz="1 0 0" />
   </joint>
   <link
-    name="komodo_$(arg komodo_id)_FL_Wheel_link">
+    name="komodo_FL_Wheel_link">
     <inertial>
       <origin
@@ -139,5 +158,5 @@
   </link>
   <joint
-    name="komodo_$(arg komodo_id)_FL_Wheel_joint"
+    name="komodo_FL_Wheel_joint"
     type="continuous">
     <origin
@@ -145,12 +164,12 @@
       rpy="-2.62229105359916E-15 6.93084604642783E-17 -1.5707963267949" />
     <parent
-      link="komodo_$(arg komodo_id)_base_link" />
-    <child
-      link="komodo_$(arg komodo_id)_FL_Wheel_link" />
+      link="komodo_base_link" />
+    <child
+      link="komodo_FL_Wheel_link" />
     <axis
       xyz="-1 0 0" />
   </joint>
   <link
-    name="komodo_$(arg komodo_id)_RR_Wheel_link">
+    name="komodo_RR_Wheel_link">
     <inertial>
       <origin
@@ -194,5 +213,5 @@
   </link>
   <joint
-    name="komodo_$(arg komodo_id)_RR_Wheel_joint"
+    name="komodo_RR_Wheel_joint"
     type="continuous">
     <origin
@@ -200,12 +219,12 @@
       rpy="2.62229105359916E-15 -1.59433090848306E-31 1.5707963267949" />
     <parent
-      link="komodo_$(arg komodo_id)_base_link" />
-    <child
-      link="komodo_$(arg komodo_id)_RR_Wheel_link" />
+      link="komodo_base_link" />
+    <child
+      link="komodo_RR_Wheel_link" />
     <axis
       xyz="1 0 0" />
   </joint>
   <link
-    name="komodo_$(arg komodo_id)_RL_Wheel_link">
+    name="komodo_RL_Wheel_link">
     <inertial>
       <origin
@@ -249,5 +268,5 @@
   </link>
   <joint
-    name="komodo_$(arg komodo_id)_RL_Wheel_joint"
+    name="komodo_RL_Wheel_joint"
     type="continuous">
     <origin
@@ -255,12 +274,12 @@
       rpy="-2.62229105359916E-15 -5.57680208627196E-32 -1.5707963267949" />
     <parent
-      link="komodo_$(arg komodo_id)_base_link" />
-    <child
-      link="komodo_$(arg komodo_id)_RL_Wheel_link" />
+      link="komodo_base_link" />
+    <child
+      link="komodo_RL_Wheel_link" />
     <axis
       xyz="-1 0 0" />
   </joint>
   <link
-    name="komodo_$(arg komodo_id)_Left_URF_link">
+    name="komodo_Left_URF_link">
     <inertial>
       <origin
@@ -302,5 +321,5 @@
   </link>
   <joint
-    name="komodo_$(arg komodo_id)_Left_URF_joint"
+    name="komodo_Left_URF_joint"
     type="fixed">
     <origin
@@ -308,12 +327,12 @@
       rpy="-2.73331335606168E-15 1.59433090848306E-31 1.5707963267949" />
     <parent
-      link="komodo_$(arg komodo_id)_base_link" />
-    <child
-      link="komodo_$(arg komodo_id)_Left_URF_link" />
+      link="komodo_base_link" />
+    <child
+      link="komodo_Left_URF_link" />
     <axis
       xyz="-1 0 0" />
   </joint>
   <link
-    name="komodo_$(arg komodo_id)_Rear_URF_link">
+    name="komodo_Rear_URF_link">
     <inertial>
       <origin
@@ -355,5 +374,5 @@
   </link>
   <joint
-    name="komodo_$(arg komodo_id)_Rear_URF_joint"
+    name="komodo_Rear_URF_joint"
     type="fixed">
     <origin
@@ -361,12 +380,12 @@
       rpy="-6.16297582203915E-33 2.73331335606168E-15 3.14159265358979" />
     <parent
-      link="komodo_$(arg komodo_id)_base_link" />
-    <child
-      link="komodo_$(arg komodo_id)_Rear_URF_link" />
+      link="komodo_base_link" />
+    <child
+      link="komodo_Rear_URF_link" />
     <axis
       xyz="-1 0 0" />
   </joint>
   <link
-    name="komodo_$(arg komodo_id)_Right_URF_link">
+    name="komodo_Right_URF_link">
     <inertial>
       <origin
@@ -408,5 +427,5 @@
   </link>
   <joint
-    name="komodo_$(arg komodo_id)_Right_URF_joint"
+    name="komodo_Right_URF_joint"
     type="fixed">
     <origin
@@ -414,12 +433,12 @@
       rpy="2.73331335606168E-15 -1.59433090848306E-31 -1.5707963267949" />
     <parent
-      link="komodo_$(arg komodo_id)_base_link" />
-    <child
-      link="komodo_$(arg komodo_id)_Right_URF_link" />
+      link="komodo_base_link" />
+    <child
+      link="komodo_Right_URF_link" />
     <axis
       xyz="-1 0 0" />
   </joint>
   <link
-    name="komodo_$(arg komodo_id)_Front_Camera_link">
+    name="komodo_Front_Camera_link">
     <inertial>
       <origin
@@ -461,5 +480,5 @@
   </link>
   <joint
-    name="komodo_$(arg komodo_id)_Front_Camera_joint"
+    name="komodo_Front_Camera_joint"
     type="fixed">
     <origin
@@ -467,12 +486,12 @@
       rpy="-1.57079632679489 -6.93084604642783E-17 -1.5707963267949" />
     <parent
-      link="komodo_$(arg komodo_id)_base_link" />
-    <child
-      link="komodo_$(arg komodo_id)_Front_Camera_link" />
+      link="komodo_base_link" />
+    <child
+      link="komodo_Front_Camera_link" />
     <axis
       xyz="0 0 1" />
   </joint>
   <link
-    name="komodo_$(arg komodo_id)_Laser_link">
+    name="komodo_Laser_link">
     <inertial>
       <origin
@@ -514,5 +533,5 @@
   </link>
   <joint
-    name="komodo_$(arg komodo_id)_Laser_joint"
+    name="komodo_Laser_joint"
     type="fixed">
     <origin
@@ -520,12 +539,12 @@
       rpy="-6.93084604642783E-17 -2.62229105359916E-15 5.55111512312578E-17" />
     <parent
-      link="komodo_$(arg komodo_id)_base_link" />
-    <child
-      link="komodo_$(arg komodo_id)_Laser_link" />
+      link="komodo_base_link" />
+    <child
+      link="komodo_Laser_link" />
     <axis
       xyz="0 0 -1" />
   </joint>
   <link
-    name="komodo_$(arg komodo_id)_Asus_Camera_link">
+    name="komodo_Asus_Camera_link">
     <inertial>
       <origin
@@ -567,5 +586,5 @@
   </link>
   <joint
-    name="komodo_$(arg komodo_id)_Asus_Camera_joint"
+    name="komodo_Asus_Camera_joint"
     type="fixed">
     <origin
@@ -573,12 +592,12 @@
       rpy="-6.93084604642783E-17 -2.62229105359916E-15 5.55111512312578E-17" />
     <parent
-      link="komodo_$(arg komodo_id)_base_link" />
-    <child
-      link="komodo_$(arg komodo_id)_Asus_Camera_link" />
+      link="komodo_base_link" />
+    <child
+      link="komodo_Asus_Camera_link" />
     <axis
       xyz="-1 0 0" />
   </joint>
   <link
-    name="komodo_$(arg komodo_id)_Arm_base_link">
+    name="komodo_Arm_base_link">
     <inertial>
       <origin
@@ -620,5 +639,5 @@
   </link>
   <joint
-    name="komodo_$(arg komodo_id)_Arm_base_joint"
+    name="komodo_Arm_base_joint"
     type="fixed">
     <origin
@@ -626,12 +645,12 @@
       rpy="3.54761842723405E-15 -3.56763412295181E-15 -3.35371649289343E-30" />
     <parent
-      link="komodo_$(arg komodo_id)_base_link" />
-    <child
-      link="komodo_$(arg komodo_id)_Arm_base_link" />
+      link="komodo_base_link" />
+    <child
+      link="komodo_Arm_base_link" />
     <axis
       xyz="0 0 1" />
   </joint>
   <link
-    name="komodo_$(arg komodo_id)_base_rotation_link">
+    name="komodo_base_rotation_link">
     <inertial>
       <origin
@@ -673,5 +692,5 @@
   </link>
   <joint
-    name="komodo_$(arg komodo_id)_base_rotation_joint"
+    name="komodo_base_rotation_joint"
     type="revolute">
     <origin
@@ -679,7 +698,7 @@
       rpy="-5.46369598732866E-16 1.34659130519145E-15 -2.1922983760752E-31" />
     <parent
-      link="komodo_$(arg komodo_id)_Arm_base_link" />
-    <child
-      link="komodo_$(arg komodo_id)_base_rotation_link" />
+      link="komodo_Arm_base_link" />
+    <child
+      link="komodo_base_rotation_link" />
     <axis
       xyz="0 0 1" />
@@ -691,5 +710,5 @@
   </joint>
   <link
-    name="komodo_$(arg komodo_id)_shoulder_link">
+    name="komodo_shoulder_link">
     <inertial>
       <origin
@@ -731,5 +750,5 @@
   </link>
   <joint
-    name="komodo_$(arg komodo_id)_shoulder_joint"
+    name="komodo_shoulder_joint"
     type="revolute">
     <origin
@@ -737,7 +756,7 @@
       rpy="-4.20159904047482E-15 -5.97509793174248E-16 9.93431320775303E-15" />
     <parent
-      link="komodo_$(arg komodo_id)_base_rotation_link" />
-    <child
-      link="komodo_$(arg komodo_id)_shoulder_link" />
+      link="komodo_base_rotation_link" />
+    <child
+      link="komodo_shoulder_link" />
     <axis
       xyz="0 1 0" />
@@ -749,5 +768,5 @@
   </joint>
   <link
-    name="komodo_$(arg komodo_id)_elbow1_link">
+    name="komodo_elbow1_link">
     <inertial>
       <origin
@@ -789,5 +808,5 @@
   </link>
   <joint
-    name="komodo_$(arg komodo_id)_elbow1_joint"
+    name="komodo_elbow1_joint"
     type="revolute">
     <origin
@@ -795,7 +814,7 @@
       rpy="1.44504380352115E-15 1.11628850952447E-06 -9.93431159466724E-15" />
     <parent
-      link="komodo_$(arg komodo_id)_shoulder_link" />
-    <child
-      link="komodo_$(arg komodo_id)_elbow1_link" />
+      link="komodo_shoulder_link" />
+    <child
+      link="komodo_elbow1_link" />
     <axis
       xyz="-0.999999999998754 0 0" />
@@ -807,5 +826,5 @@
   </joint>
   <link
-    name="komodo_$(arg komodo_id)_elbow2_link">
+    name="komodo_elbow2_link">
     <inertial>
       <origin
@@ -847,5 +866,5 @@
   </link>
   <joint
-    name="komodo_$(arg komodo_id)_elbow2_joint"
+    name="komodo_elbow2_joint"
     type="revolute">
     <origin
@@ -853,7 +872,7 @@
       rpy="-4.51048856041191E-16 3.35869632765754E-16 0" />
     <parent
-      link="komodo_$(arg komodo_id)_elbow1_link" />
-    <child
-      link="komodo_$(arg komodo_id)_elbow2_link" />
+      link="komodo_elbow1_link" />
+    <child
+      link="komodo_elbow2_link" />
     <axis
       xyz="0 1 0" />
@@ -865,5 +884,5 @@
   </joint>
   <link
-    name="komodo_$(arg komodo_id)_wrist_link">
+    name="komodo_wrist_link">
     <inertial>
       <origin
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