Commit message: Removed 'Komodo_id' link prefix, added smplified meshes for collision calculations

File: ric_description/komodo/komodo.xacro (robot description, xacro)
@@ -4,8 +4,8 @@
 <!-- Dummy inertia link & Joint -->
   <link
-    name="komodo_dummy_link">
+    name="dummy_link">
 </link>
   <joint
-    name="komodo_dummy_joint"
+    name="dummy_joint"
     type="fixed">
     <origin
@@ -13,7 +13,7 @@
       rpy="0 0 0" />
     <parent
-      link="komodo_dummy_link" />
-    <child
-      link="komodo_base_link" />
+      link="dummy_link" />
+    <child
+      link="base_link" />
     <axis
       xyz="0 0 0" />
@@ -21,5 +21,5 @@
 <!-- Dummy link & node -->
   <link
-    name="komodo_base_link">
+    name="base_link">
     <inertial>
       <origin
@@ -61,5 +61,5 @@
   </link>
   <link
-    name="komodo_FR_Wheel_link">
+    name="FR_Wheel_link">
     <inertial>
       <origin
@@ -103,5 +103,5 @@
   </link>
   <joint
-    name="komodo_FR_Wheel_joint"
+    name="FR_Wheel_joint"
     type="continuous">
     <origin
@@ -109,12 +109,12 @@
       rpy="2.62229105359916E-15 6.9308460464278E-17 1.5707963267949" />
     <parent
-      link="komodo_base_link" />
-    <child
-      link="komodo_FR_Wheel_link" />
+      link="base_link" />
+    <child
+      link="FR_Wheel_link" />
     <axis
       xyz="1 0 0" />
   </joint>
   <link
-    name="komodo_FL_Wheel_link">
+    name="FL_Wheel_link">
     <inertial>
       <origin
@@ -158,5 +158,5 @@
   </link>
   <joint
-    name="komodo_FL_Wheel_joint"
+    name="FL_Wheel_joint"
     type="continuous">
     <origin
@@ -164,12 +164,12 @@
       rpy="-2.62229105359916E-15 6.93084604642783E-17 -1.5707963267949" />
     <parent
-      link="komodo_base_link" />
-    <child
-      link="komodo_FL_Wheel_link" />
+      link="base_link" />
+    <child
+      link="FL_Wheel_link" />
     <axis
       xyz="-1 0 0" />
   </joint>
   <link
-    name="komodo_RR_Wheel_link">
+    name="RR_Wheel_link">
     <inertial>
       <origin
@@ -213,5 +213,5 @@
   </link>
   <joint
-    name="komodo_RR_Wheel_joint"
+    name="RR_Wheel_joint"
     type="continuous">
     <origin
@@ -219,12 +219,12 @@
       rpy="2.62229105359916E-15 -1.59433090848306E-31 1.5707963267949" />
     <parent
-      link="komodo_base_link" />
-    <child
-      link="komodo_RR_Wheel_link" />
+      link="base_link" />
+    <child
+      link="RR_Wheel_link" />
     <axis
       xyz="1 0 0" />
   </joint>
   <link
-    name="komodo_RL_Wheel_link">
+    name="RL_Wheel_link">
     <inertial>
       <origin
@@ -268,5 +268,5 @@
   </link>
   <joint
-    name="komodo_RL_Wheel_joint"
+    name="RL_Wheel_joint"
     type="continuous">
     <origin
@@ -274,12 +274,12 @@
       rpy="-2.62229105359916E-15 -5.57680208627196E-32 -1.5707963267949" />
     <parent
-      link="komodo_base_link" />
-    <child
-      link="komodo_RL_Wheel_link" />
+      link="base_link" />
+    <child
+      link="RL_Wheel_link" />
     <axis
       xyz="-1 0 0" />
   </joint>
   <link
-    name="komodo_Left_URF_link">
+    name="Left_URF_link">
     <inertial>
       <origin
@@ -321,5 +321,5 @@
   </link>
   <joint
-    name="komodo_Left_URF_joint"
+    name="Left_URF_joint"
     type="fixed">
     <origin
@@ -327,12 +327,12 @@
       rpy="-2.73331335606168E-15 1.59433090848306E-31 1.5707963267949" />
     <parent
-      link="komodo_base_link" />
-    <child
-      link="komodo_Left_URF_link" />
+      link="base_link" />
+    <child
+      link="Left_URF_link" />
     <axis
       xyz="-1 0 0" />
   </joint>
   <link
-    name="komodo_Rear_URF_link">
+    name="Rear_URF_link">
     <inertial>
       <origin
@@ -374,5 +374,5 @@
   </link>
   <joint
-    name="komodo_Rear_URF_joint"
+    name="Rear_URF_joint"
     type="fixed">
     <origin
@@ -380,12 +380,12 @@
       rpy="-6.16297582203915E-33 2.73331335606168E-15 3.14159265358979" />
     <parent
-      link="komodo_base_link" />
-    <child
-      link="komodo_Rear_URF_link" />
+      link="base_link" />
+    <child
+      link="Rear_URF_link" />
     <axis
       xyz="-1 0 0" />
   </joint>
   <link
-    name="komodo_Right_URF_link">
+    name="Right_URF_link">
     <inertial>
       <origin
@@ -427,5 +427,5 @@
   </link>
   <joint
-    name="komodo_Right_URF_joint"
+    name="Right_URF_joint"
     type="fixed">
     <origin
@@ -433,12 +433,12 @@
       rpy="2.73331335606168E-15 -1.59433090848306E-31 -1.5707963267949" />
     <parent
-      link="komodo_base_link" />
-    <child
-      link="komodo_Right_URF_link" />
+      link="base_link" />
+    <child
+      link="Right_URF_link" />
     <axis
       xyz="-1 0 0" />
   </joint>
   <link
-    name="komodo_Front_Camera_link">
+    name="Front_Camera_link">
     <inertial>
       <origin
@@ -480,5 +480,5 @@
   </link>
   <joint
-    name="komodo_Front_Camera_joint"
+    name="Front_Camera_joint"
     type="fixed">
     <origin
@@ -486,12 +486,12 @@
       rpy="-1.57079632679489 -6.93084604642783E-17 -1.5707963267949" />
     <parent
-      link="komodo_base_link" />
-    <child
-      link="komodo_Front_Camera_link" />
+      link="base_link" />
+    <child
+      link="Front_Camera_link" />
     <axis
       xyz="0 0 1" />
   </joint>
   <link
-    name="komodo_Laser_link">
+    name="Laser_link">
     <inertial>
       <origin
@@ -533,5 +533,5 @@
   </link>
   <joint
-    name="komodo_Laser_joint"
+    name="Laser_joint"
     type="fixed">
     <origin
@@ -539,12 +539,12 @@
       rpy="-6.93084604642783E-17 -2.62229105359916E-15 5.55111512312578E-17" />
     <parent
-      link="komodo_base_link" />
-    <child
-      link="komodo_Laser_link" />
+      link="base_link" />
+    <child
+      link="Laser_link" />
     <axis
       xyz="0 0 -1" />
   </joint>
   <link
-    name="komodo_Asus_Camera_link">
+    name="Asus_Camera_link">
     <inertial>
       <origin
@@ -586,5 +586,5 @@
   </link>
   <joint
-    name="komodo_Asus_Camera_joint"
+    name="Asus_Camera_joint"
     type="fixed">
     <origin
@@ -592,12 +592,12 @@
       rpy="-6.93084604642783E-17 -2.62229105359916E-15 5.55111512312578E-17" />
     <parent
-      link="komodo_base_link" />
-    <child
-      link="komodo_Asus_Camera_link" />
+      link="base_link" />
+    <child
+      link="Asus_Camera_link" />
     <axis
       xyz="-1 0 0" />
   </joint>
   <link
-    name="komodo_Arm_base_link">
+    name="Arm_base_link">
     <inertial>
       <origin
@@ -639,5 +639,5 @@
   </link>
   <joint
-    name="komodo_Arm_base_joint"
+    name="Arm_base_joint"
     type="fixed">
     <origin
@@ -645,12 +645,12 @@
       rpy="3.54761842723405E-15 -3.56763412295181E-15 -3.35371649289343E-30" />
     <parent
-      link="komodo_base_link" />
-    <child
-      link="komodo_Arm_base_link" />
+      link="base_link" />
+    <child
+      link="Arm_base_link" />
     <axis
       xyz="0 0 1" />
   </joint>
   <link
-    name="komodo_base_rotation_link">
+    name="base_rotation_link">
     <inertial>
       <origin
@@ -687,10 +687,10 @@
       <geometry>
         <mesh
-          filename="package://ric_description/komodo/meshes/base_rotation_link.STL" />
-      </geometry>
-    </collision>
-  </link>
-  <joint
-    name="komodo_base_rotation_joint"
+          filename="package://ric_description/komodo/meshes/col_base_rotation_link.STL" />
+      </geometry>
+    </collision>
+  </link>
+  <joint
+    name="base_rotation_joint"
     type="revolute">
     <origin
@@ -698,7 +698,7 @@
       rpy="-5.46369598732866E-16 1.34659130519145E-15 -2.1922983760752E-31" />
     <parent
-      link="komodo_Arm_base_link" />
-    <child
-      link="komodo_base_rotation_link" />
+      link="Arm_base_link" />
+    <child
+      link="base_rotation_link" />
     <axis
       xyz="0 0 1" />
@@ -710,5 +710,5 @@
   </joint>
   <link
-    name="komodo_shoulder_link">
+    name="shoulder_link">
     <inertial>
       <origin
@@ -745,10 +745,10 @@
       <geometry>
         <mesh
-          filename="package://ric_description/komodo/meshes/shoulder_link.STL" />
-      </geometry>
-    </collision>
-  </link>
-  <joint
-    name="komodo_shoulder_joint"
+          filename="package://ric_description/komodo/meshes/col_shoulder_link.STL" />
+      </geometry>
+    </collision>
+  </link>
+  <joint
+    name="shoulder_joint"
     type="revolute">
     <origin
@@ -756,7 +756,7 @@
       rpy="-4.20159904047482E-15 -5.97509793174248E-16 9.93431320775303E-15" />
     <parent
-      link="komodo_base_rotation_link" />
-    <child
-      link="komodo_shoulder_link" />
+      link="base_rotation_link" />
+    <child
+      link="shoulder_link" />
     <axis
       xyz="0 1 0" />
@@ -768,5 +768,5 @@
   </joint>
   <link
-    name="komodo_elbow1_link">
+    name="elbow1_link">
     <inertial>
       <origin
@@ -803,10 +803,10 @@
       <geometry>
         <mesh
-          filename="package://ric_description/komodo/meshes/elbow1_link.STL" />
-      </geometry>
-    </collision>
-  </link>
-  <joint
-    name="komodo_elbow1_joint"
+          filename="package://ric_description/komodo/meshes/col_elbow1_link.STL" />
+      </geometry>
+    </collision>
+  </link>
+  <joint
+    name="elbow1_joint"
     type="revolute">
     <origin
@@ -814,7 +814,7 @@
       rpy="1.44504380352115E-15 1.11628850952447E-06 -9.93431159466724E-15" />
     <parent
-      link="komodo_shoulder_link" />
-    <child
-      link="komodo_elbow1_link" />
+      link="shoulder_link" />
+    <child
+      link="elbow1_link" />
     <axis
       xyz="-0.999999999998754 0 0" />
@@ -826,5 +826,5 @@
   </joint>
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
Commit message: Included simplified meshes, rviz config files for both single and multi launch with all sensors and added front camera

File: ric_description/komodo/komodo.xacro (robot description, xacro)
@@ -42,5 +42,5 @@
       <geometry>
         <mesh
-          filename="package://ric_description/komodo/meshes/base_link.STL" />
+          filename="package://ric_description/komodo/meshes/col_base_link.STL" />
       </geometry>
       <material
@@ -56,5 +56,5 @@
       <geometry>
         <mesh
-          filename="package://ric_description/komodo/meshes/base_link.STL" />
+          filename="package://ric_description/komodo/meshes/col_base_link.STL" />
       </geometry>
     </collision>
@@ -458,5 +458,5 @@
       <origin
         xyz="0 0 0"
-        rpy="0 0 0" />
+        rpy="-1.57079632649567 1.57079632649567 -1.57079632649567" />
       <geometry>
         <mesh
@@ -472,5 +472,5 @@
       <origin
         xyz="0 0 0"
-        rpy="0 0 0" />
+        rpy="1.57 0 0" />
       <geometry>
         <mesh
@@ -484,5 +484,5 @@
     <origin
       xyz="0.262250027816762 0.0875000000000051 0.100000000000001"
-      rpy="-1.57079632679489 -6.93084604642783E-17 -1.5707963267949" />
+      rpy="0 0 0" />
     <parent
       link="base_link" />
@@ -672,6 +672,8 @@
         rpy="0 0 0" />
       <geometry>
-        <mesh
-          filename="package://ric_description/komodo/meshes/base_rotation_link.STL" />
+        <!--mesh
+          filename="package://ric_description/komodo/meshes/base_rotation_link.STL" /-->
+	<mesh
+          filename="package://ric_description/komodo/meshes/col_base_rotation_link.STL" />
       </geometry>
       <material
@@ -687,5 +689,5 @@
       <geometry>
         <mesh
-          filename="package://ric_description/komodo/meshes/base_rotation_link.STL" />
+          filename="package://ric_description/komodo/meshes/col_base_rotation_link.STL" /> <!-- Simplified -->
       </geometry>
     </collision>
@@ -731,5 +733,5 @@
       <geometry>
         <mesh
-          filename="package://ric_description/komodo/meshes/shoulder_link.STL" />
+          filename="package://ric_description/komodo/meshes/col_shoulder_link.STL" /> <!-- Simplified -->
       </geometry>
       <material
@@ -745,5 +747,5 @@
       <geometry>
         <mesh
-          filename="package://ric_description/komodo/meshes/shoulder_link.STL" />
+          filename="package://ric_description/komodo/meshes/col_shoulder_link.STL" /> <!-- Simplified -->
       </geometry>
     </collision>
@@ -789,5 +791,5 @@
       <geometry>
         <mesh
-          filename="package://ric_description/komodo/meshes/elbow1_link.STL" />
+          filename="package://ric_description/komodo/meshes/col_elbow1_link.STL" />  <!-- Simplified -->
       </geometry>
       <material
@@ -803,5 +805,5 @@
       <geometry>
         <mesh
-          filename="package://ric_description/komodo/meshes/elbow1_link.STL" />
+         filename="package://ric_description/komodo/meshes/col_elbow1_link.STL" />  <!-- Simplified -->
       </geometry>
     </collision>
@@ -847,5 +849,5 @@
       <geometry>
         <mesh
-          filename="package://ric_description/komodo/meshes/elbow2_link.STL" />
+           filename="package://ric_description/komodo/meshes/col_elbow2_link.STL" />  <!-- Simplified -->
       </geometry>
       <material
@@ -861,5 +863,5 @@
       <geometry>
         <mesh
-          filename="package://ric_description/komodo/meshes/elbow2_link.STL" />
+          filename="package://ric_description/komodo/meshes/col_elbow2_link.STL" />  <!-- Simplified -->
       </geometry>
     </collision>
@@ -905,5 +907,5 @@
       <geometry>
         <mesh
-          filename="package://ric_description/komodo/meshes/wrist_link.STL" />
+        filename="package://ric_description/komodo/meshes/col_wrist_link.STL" />  <!-- Simplified -->
       </geometry>
       <material
@@ -919,5 +921,5 @@
       <geometry>
         <mesh
-          filename="package://ric_description/komodo/meshes/wrist_link.STL" />
+          filename="package://ric_description/komodo/meshes/col_wrist_link.STL" />  <!-- Simplified -->
       </geometry>
     </collision>
@@ -963,5 +965,5 @@
       <geometry>
         <mesh
-          filename="package://ric_description/komodo/meshes/left_finger_link.STL" />
+          filename="package://ric_description/komodo/meshes/col_left_finger_link.STL" />  <!-- Simplified -->
       </geometry>
       <material
@@ -977,5 +979,5 @@
       <geometry>
         <mesh
-          filename="package://ric_description/komodo/meshes/left_finger_link.STL" />
+          filename="package://ric_description/komodo/meshes/col_left_finger_link.STL" />  <!-- Simplified -->
       </geometry>
     </collision>
@@ -1021,5 +1023,5 @@
       <geometry>
         <mesh
-          filename="package://ric_description/komodo/meshes/right_finger_link.STL" />
+          filename="package://ric_description/komodo/meshes/col_right_finger_link.STL" />  <!-- Simplified -->
       </geometry>
       <material
@@ -1035,5 +1037,5 @@
       <geometry>
         <mesh
-          filename="package://ric_description/komodo/meshes/right_finger_link.STL" />
+           filename="package://ric_description/komodo/meshes/col_right_finger_link.STL" />  <!-- Simplified -->
       </geometry>
     </collision>
@@ -1355,5 +1357,5 @@
       <visualize>false</visualize>
       <update_rate>30.0</update_rate>
-      <camera name="arm">
+      <camera name="arm_camera">
         <horizontal_fov>2.0</horizontal_fov>
         <image>
@@ -1364,15 +1366,47 @@
         <clip>
           <near>0.02</near>
-          <far>300</far>
+          <far>9</far>
         </clip>
       </camera>
       <plugin name="camera_controller" filename="libgazebo_ros_camera.so">
         <alwaysOn>true</alwaysOn>
-        <updateRate>40.0</updateRate>
-        <robotNamespace>komodo_$(arg komodo_id)_Arm_Camera_link</robotNamespace>
-        <cameraName>/komodo_$(arg komodo_id)/arm_camera</cameraName>
-        <imageTopicName>/komodo_$(arg komodo_id)/arm_camera/image_raw</imageTopicName>
-        <cameraInfoTopicName>/komodo_$(arg komodo_id)/arm_camera/camera_info</cameraInfoTopicName>
-        <!--frameName>Arm_Camera_link</frameName-->
+        <robotNamespace>komodo_$(arg komodo_id)</robotNamespace>
+        <cameraName>arm_camera</cameraName>
+        <imageTopicName>arm_camera/image_raw</imageTopicName>
+        <cameraInfoTopicName>arm_camera/camera_info</cameraInfoTopicName>
+        <frameName>Arm_Camera_link</frameName>
+        <hackBaseline>0.07</hackBaseline>
+        <distortionK1>0.0</distortionK1>
+        <distortionK2>0.0</distortionK2>
+        <distortionK3>0.0</distortionK3>
+        <distortionT1>0.0</distortionT1>
+        <distortionT2>0.0</distortionT2>
+      </plugin>
+    </sensor>
+  </gazebo>
+<!-- front camera -->
+  <gazebo reference="Front_Camera_link">
+    <sensor type="camera" name="camera2">
+      <visualize>false</visualize>
+      <update_rate>30.0</update_rate>
+      <camera name="Front_Camera">
+        <horizontal_fov>2.0</horizontal_fov>
+        <image>
+          <width>1800</width>
+          <height>1800</height>
+          <format>R8G8B8</format>
+        </image>
+        <clip>
+          <near>0.02</near>
+          <far>9</far>
+        </clip>
+      </camera>
+      <plugin name="camera_controller" filename="libgazebo_ros_camera.so">
+        <alwaysOn>true</alwaysOn>
+        <robotNamespace>komodo_$(arg komodo_id)</robotNamespace>
+        <cameraName>Front_Camera</cameraName>
+        <imageTopicName>Front_Camera/image_raw</imageTopicName>
+        <cameraInfoTopicName>Front_Camera/camera_info</cameraInfoTopicName>
+        <frameName>Front_Camera_link</frameName>
         <hackBaseline>0.07</hackBaseline>
         <distortionK1>0.0</distortionK1>
@@ -1386,73 +1420,40 @@
 <!-- Asus camera  - Gazebo -->
 <gazebo reference="Asus_Camera_link">
-<sensor type="depth" name="Asus_Camera_link">
-<pose>0 0 0 0 0 0</pose>
-<visualize>true</visualize>
-<update_rate>20</update_rate>
-<camera>
-<horizontal_fov>2.0</horizontal_fov>
-<image>
-<format>R8G8B8</format>
-<width>640</width>
-<height>480</height>
-</image>
-<clip>
-<near>0.5</near>
-<far>9</far>
-</clip>
-</camera>
-<plugin name="Asus_Camera_link_camera_controller" filename="libgazebo_ros_openni_kinect.so">
-<alwaysOn>true</alwaysOn>
-<updateRate>20</updateRate>
-<cameraName>komodo_Asus_Camera</cameraName>
-<!--robotNamespace>/komodo_$(arg komodo_id)</robotNamespace-->
-<imageTopicName>/komodo_$(arg komodo_id)/komodo_Asus_Camera/rgb/image_raw</imageTopicName>
-<cameraInfoTopicName>/komodo_$(arg komodo_id)/komodo_Asus_Camera/rgb/camera_info</cameraInfoTopicName>
-<depthImageTopicName>/komodo_$(arg komodo_id)/komodo_Asus_Camera/depth/image_raw</depthImageTopicName>
-<depthImageCameraInfoTopicName>/komodo_$(arg komodo_id)/komodo_Asus_Camera/depth/camera_info</depthImageCameraInfoTopicName>
-<pointCloudTopicName>/komodo_$(arg komodo_id)/komodo_Asus_Camera/depth/points</pointCloudTopicName>
-<pointCloudCutoff>0.4</pointCloudCutoff>
-<frameName>/Asus_Camera_link</frameName>
-<distortion_k1>0.0</distortion_k1>
-<distortion_k2>0.0</distortion_k2>
-<distortion_k3>0.0</distortion_k3>
-<distortion_t1>0.0</distortion_t1>
-<distortion_t2>0.0</distortion_t2>
-</plugin>
-</sensor>
+	<sensor type="depth" name="Asus_Camera_link">
+	  <pose>0 0 0 0 0 0</pose>
+	  <visualize>true</visualize>
+          <update_rate>20</update_rate>
+	 	<camera>
+		<horizontal_fov>2.0</horizontal_fov>
+			<image>
+			<format>R8G8B8</format>
+			<width>640</width>
+			<height>480</height>
+			</image>
+		<clip>
+		<near>0.5</near>
+		<far>9</far>
+		</clip>
+		</camera>
+	<plugin name="Asus_Camera_link_camera_controller" filename="libgazebo_ros_openni_kinect.so">
+	<alwaysOn>true</alwaysOn>
+	<updateRate>20</updateRate>
+	<cameraName>komodo_Asus_Camera</cameraName>
+	<!--robotNamespace>/komodo_$(arg komodo_id)</robotNamespace-->
+	<imageTopicName>/komodo_$(arg komodo_id)/komodo_Asus_Camera/rgb/image_raw</imageTopicName>
+	<cameraInfoTopicName>/komodo_$(arg komodo_id)/komodo_Asus_Camera/rgb/camera_info</cameraInfoTopicName>
+	<depthImageTopicName>/komodo_$(arg komodo_id)/komodo_Asus_Camera/depth/image_raw</depthImageTopicName>
+	<depthImageCameraInfoTopicName>/komodo_$(arg komodo_id)/komodo_Asus_Camera/depth/camera_info</depthImageCameraInfoTopicName>
+	<pointCloudTopicName>/komodo_$(arg komodo_id)/komodo_Asus_Camera/depth/points</pointCloudTopicName>
+	<pointCloudCutoff>0.4</pointCloudCutoff>
+	<frameName>/Asus_Camera_link</frameName>
+	<distortion_k1>0.0</distortion_k1>
+	<distortion_k2>0.0</distortion_k2>
+	<distortion_k3>0.0</distortion_k3>
+	<distortion_t1>0.0</distortion_t1>
+	<distortion_t2>0.0</distortion_t2>
+	</plugin>
+    </sensor>
 </gazebo>
-<!-- ASUS Xtion PRO camera for simulation
-      <gazebo reference="komodo_Asus_Camera_link">
-        <sensor type="depth" name="komodo_Asus_Camera_link">
-          <update_rate>20</update_rate>
-          <camera>
-            <horizontal_fov>${62.8 * M_PI/180.0}</horizontal_fov>
-            <image>
-              <format>R8G8B8</format>
-              <width>640</width>
-              <height>480</height>
-            </image>
-            <clip>
-              <near>0.5</near>
-              <far>9</far>
-            </clip>
-          </camera>
-          <plugin name="komodo_Asus_Camera_link_camera_controller" filename="libgazebo_ros_openni_kinect.so">
-            <alwaysOn>true</alwaysOn>
-            <updateRate>20</updateRate>
-            <imageTopicName>komodo_Asus_Camera_link/rgb/image_raw</imageTopicName>
-            <cameraInfoTopicName>komodo_Asus_Camera_link/rgb/camera_info</cameraInfoTopicName>
-            <depthImageTopicName>komodo_Asus_Camera_link/depth/image_raw</depthImageTopicName>
-            <depthImageCameraInfoTopicName>komodo_Asus_Camera_link/depth/camera_info</depthImageCameraInfoTopicName>
-            <pointCloudTopicName>komodo_Asus_Camera_link/depth/points</pointCloudTopicName>
-            <frameName>komodo_Asus_Camera_link</frameName>
-            <distortion_k1>0.0</distortion_k1>
-            <distortion_k2>0.0</distortion_k2>
-            <distortion_k3>0.0</distortion_k3>
-            <distortion_t1>0.0</distortion_t1>
-            <distortion_t2>0.0</distortion_t2>
-          </plugin>
-        </sensor>
-      </gazebo -->
   <!-- hokuyo -->
   <gazebo reference="Laser_link">
