Commit message: komodo xacro

File: ric_description/komodo/komodo_no_arm_no_plugins2.xacro (robot description, xacro)
@@ -579,518 +579,4 @@
   </joint>
   <link
-    name="Arm_base_link">
-    <inertial>
-      <origin
-        xyz="-0.0168723530982394 -5.23224904403848E-05 0.038112696778507"
-        rpy="0 0 0" />
-      <mass
-        value="1.08982930885161" />
-      <inertia
-        ixx="0.00311458437968986"
-        ixy="-7.0610782277189E-06"
-        ixz="-0.000262941654993437"
-        iyy="0.00855106134499406"
-        iyz="1.00391927392762E-06"
-        izz="0.0104177337437887" />
-    </inertial>
-    <visual>
-      <origin
-        xyz="0 0 0"
-        rpy="0 0 0" />
-      <geometry>
-        <mesh
-          filename="package://ric_description/komodo/meshes/Arm_base_link.STL" />
-      </geometry>
-      <material
-        name="">
-        <color
-          rgba="0.4 0.4 0.4 1" />
-      </material>
-    </visual>
-    <collision>
-      <origin
-        xyz="0 0 0"
-        rpy="0 0 0" />
-      <geometry>
-        <mesh
-          filename="package://ric_description/komodo/meshes/Arm_base_link.STL" />
-      </geometry>
-    </collision>
-  </link>
-  <joint
-    name="Arm_base_joint"
-    type="fixed">
-    <origin
-      xyz="-0.112249972183238 0 0.167160698455407"
-      rpy="3.54761842723405E-15 -3.56763412295181E-15 -3.35371649289343E-30" />
-    <parent
-      link="base_link" />
-    <child
-      link="Arm_base_link" />
-    <axis
-      xyz="0 0 1" />
-  </joint>
-  <link
-    name="base_rotation_link">
-    <inertial>
-      <origin
-        xyz="-1.11022302462516E-16 -7.80223872637444E-17 0.0660708417371112"
-        rpy="0 0 0" />
-      <mass
-        value="1.4054258533062" />
-      <inertia
-        ixx="0.00159425912810341"
-        ixy="-8.40269196653518E-08"
-        ixz="-1.60925604895535E-19"
-        iyy="0.000605522001732049"
-        iyz="-6.08768470792684E-19"
-        izz="0.00123388334665811" />
-    </inertial>
-    <visual>
-      <origin
-        xyz="0 0 0"
-        rpy="0 0 0" />
-      <geometry>
-        <!--mesh
-          filename="package://ric_description/komodo/meshes/base_rotation_link.STL" /-->
-	<mesh
-          filename="package://ric_description/komodo/meshes/col_base_rotation_link.STL" />
-      </geometry>
-      <material
-        name="">
-        <color
-          rgba="0.3 0.3 0.3 1" />
-      </material>
-    </visual>
-    <collision>
-      <origin
-        xyz="0 0 0"
-        rpy="0 0 0" />
-      <geometry>
-        <mesh
-          filename="package://ric_description/komodo/meshes/col_base_rotation_link.STL" /> <!-- Simplified -->
-      </geometry>
-    </collision>
-  </link>
-  <joint
-    name="base_rotation_joint"
-    type="revolute">
-    <origin
-      xyz="-0.096277996026178 0 0.0549000000000002"
-      rpy="-5.46369598732866E-16 1.34659130519145E-15 -2.1922983760752E-31" />
-    <parent
-      link="Arm_base_link" />
-    <child
-      link="base_rotation_link" />
-    <axis
-      xyz="0 0 1" />
-    <limit
-      lower="-3.14"
-      upper="3.14"
-      effort="10"
-      velocity="0" />
-  </joint>
-  <link
-    name="shoulder_link">
-    <inertial>
-      <origin
-        xyz="-4.66231481405233E-06 -9.82289126283389E-05 0.0772888499682157"
-        rpy="0 0 0" />
-      <mass
-        value="0.191480823048406" />
-      <inertia
-        ixx="0.00107301595696304"
-        ixy="-2.9789063890745E-07"
-        ixz="-2.01216953964121E-08"
-        iyy="0.000975953125213584"
-        iyz="-1.19601921452086E-06"
-        izz="0.000217659789393094" />
-    </inertial>
-    <visual>
-      <origin
-        xyz="0 0 0"
-        rpy="0 0 0" />
-      <geometry>
-        <mesh
-          filename="package://ric_description/komodo/meshes/col_shoulder_link.STL" /> <!-- Simplified -->
-      </geometry>
-      <material
-        name="">
-        <color
-          rgba="0.4 0.4 0.4 1" />
-      </material>
-    </visual>
-    <collision>
-      <origin
-        xyz="0 0 0"
-        rpy="0 0 0" />
-      <geometry>
-        <mesh
-          filename="package://ric_description/komodo/meshes/col_shoulder_link.STL" /> <!-- Simplified -->
-      </geometry>
-    </collision>
-  </link>
-  <joint
-    name="shoulder_joint"
-    type="revolute">
-    <origin
-      xyz="0 0 0.0834999999999999"
-      rpy="-4.20159904047482E-15 -5.97509793174248E-16 9.93431320775303E-15" />
-    <parent
-      link="base_rotation_link" />
-    <child
-      link="shoulder_link" />
-    <axis
-      xyz="0 1 0" />
-    <limit
-      lower="-1.57"
-      upper="1.57"
-      effort="2000"
-      velocity="0" />
-  </joint>
-  <link
-    name="elbow1_link">
-    <inertial>
-      <origin
-        xyz="3.38561240652013E-05 2.66604610292575E-06 0.0239321015909688"
-        rpy="0 0 0" />
-      <mass
-        value="0.759959116000226" />
-      <inertia
-        ixx="0.0011156254663426"
-        ixy="3.16193221175592E-07"
-        ixz="2.89169705133133E-06"
-        iyy="0.00114606034071406"
-        iyz="-8.11914906919631E-08"
-        izz="0.000237163435713384" />
-    </inertial>
-    <visual>
-      <origin
-        xyz="0 0 0"
-        rpy="0 0 0" />
-      <geometry>
-        <mesh
-          filename="package://ric_description/komodo/meshes/col_elbow1_link.STL" />  <!-- Simplified -->
-      </geometry>
-      <material
-        name="">
-        <color
-          rgba="0.3 0.3 0.3 1" />
-      </material>
-    </visual>
-    <collision>
-      <origin
-        xyz="0 0 0"
-        rpy="0 0 0" />
-      <geometry>
-        <mesh
-         filename="package://ric_description/komodo/meshes/col_elbow1_link.STL" />  <!-- Simplified -->
-      </geometry>
-    </collision>
-  </link>
-  <joint
-    name="elbow1_joint"
-    type="revolute">
-    <origin
-      xyz="0 -0.000251155668932789 0.266305434894181"
-      rpy="1.44504380352115E-15 1.11628850952447E-06 -9.93431159466724E-15" />
-    <parent
-      link="shoulder_link" />
-    <child
-      link="elbow1_link" />
-    <axis
-      xyz="-0.999999999998754 0 0" />
-    <limit
-      lower="-3.14"
-      upper="3.14"
-      effort="100"
-      velocity="0" />
-  </joint>
-  <link
-    name="elbow2_link">
-    <inertial>
-      <origin
-        xyz="-2.29085121194481E-05 -0.000512185919169572 0.0885118786028204"
-        rpy="0 0 0" />
-      <mass
-        value="1.12138857800426" />
-      <inertia
-        ixx="0.0011156254663426"
-        ixy="3.04261287700186E-07"
-        ixz="-1.22468079415109E-06"
-        iyy="0.0110437302875007"
-        iyz="-7.91547787630536E-05"
-        izz="0.000331598270284794" />
-    </inertial>
-    <visual>
-      <origin
-        xyz="0 0 0"
-        rpy="0 0 0" />
-      <geometry>
-        <mesh
-           filename="package://ric_description/komodo/meshes/col_elbow2_link.STL" />  <!-- Simplified -->
-      </geometry>
-      <material
-        name="">
-        <color
-          rgba="0.4 0.4 0.4 1" />
-      </material>
-    </visual>
-    <collision>
-      <origin
-        xyz="0 0 0"
-        rpy="0 0 0" />
-      <geometry>
-        <mesh
-          filename="package://ric_description/komodo/meshes/col_elbow2_link.STL" />  <!-- Simplified -->
-      </geometry>
-    </collision>
-  </link>
-  <joint
-    name="elbow2_joint"
-    type="revolute">
-    <origin
-      xyz="0 0 0.223999999999899"
-      rpy="-4.51048856041191E-16 3.35869632765754E-16 0" />
-    <parent
-      link="elbow1_link" />
-    <child
-      link="elbow2_link" />
-    <axis
-      xyz="0 1 0" />
-    <limit
-      lower="-3.14"
-      upper="3.14"
-      effort="10"
-      velocity="0" />
-  </joint>
-  <link
-    name="wrist_link">
-    <inertial>
-      <origin
-        xyz="0 0 0"
-        rpy="0 0 0" />
-      <mass
-        value="0.717337417215465" />
-      <inertia
-        ixx="0.000486392340366094"
-        ixy="4.20757000035677E-12"
-        ixz="-3.91843889020299E-06"
-        iyy="0.000211170064630335"
-        iyz="2.79335159568522E-12"
-        izz="0.000437528795624211" />
-    </inertial>
-    <visual>
-      <origin
-        xyz="0 0 0"
-        rpy="0 0 0" />
-      <geometry>
-        <mesh
-        filename="package://ric_description/komodo/meshes/col_wrist_link.STL" />  <!-- Simplified -->
-      </geometry>
-      <material
-        name="">
-        <color
-          rgba="0.4 0.4 0.4 1" />
-      </material>
-    </visual>
-    <collision>
-      <origin
-        xyz="0 0 0"
-        rpy="0 0 0" />
-      <geometry>
-        <mesh
-          filename="package://ric_description/komodo/meshes/col_wrist_link.STL" />  <!-- Simplified -->
-      </geometry>
-    </collision>
-  </link>
-  <joint
-    name="wrist_joint"
-    type="revolute">
-    <origin
-      xyz="0.0137 0 0.244749999999997"
-      rpy="0 0 0" />
-    <parent
-      link="elbow2_link" />
-    <child
-      link="wrist_link" />
-    <axis
-      xyz="0 0 0.999999999998754" />
-    <limit
-      lower="-3.14"
-      upper="3.14"
-      effort="10"
-      velocity="0" />
-  </joint>
-  <link
-    name="left_finger_link">
-    <inertial>
-      <origin
-        xyz="-6.10622663543836E-16 0.0205697573116852 0.0301832532936965"
-        rpy="0 0 0" />
-      <mass
-        value="0.0111981711598485" />
-      <inertia
-        ixx="0.000486392340366094"
-        ixy="4.20757000035677E-12"
-        ixz="-3.91843889020299E-06"
-        iyy="0.000211170064630335"
-        iyz="2.79335159568522E-12"
-        izz="0.000437528795624211" />
-    </inertial>
-    <visual>
-      <origin
-        xyz="0 0 0"
-        rpy="0 0 0" />
-      <geometry>
-        <mesh
-          filename="package://ric_description/komodo/meshes/col_left_finger_link.STL" />  <!-- Simplified -->
-      </geometry>
-      <material
-        name="">
-        <color
-          rgba="0.4 0.4 0.4 1" />
-      </material>
-    </visual>
-    <collision>
-      <origin
-        xyz="0 0 0"
-        rpy="0 0 0" />
-      <geometry>
-        <mesh
-          filename="package://ric_description/komodo/meshes/col_left_finger_link.STL" />  <!-- Simplified -->
-      </geometry>
-    </collision>
-  </link>
-  <joint
-    name="left_finger_joint"
-    type="revolute">
-    <origin
-      xyz="-0.000250000000000111 0.021 0.0422500000000001"
-      rpy="2.85979682697881E-15 1.01870746742143E-16 3.19235832636806E-21" />
-    <parent
-      link="wrist_link" />
-    <child
-      link="left_finger_link" />
-    <axis
-      xyz="1 0 0" />
-    <limit
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