Commit message: jta updates

File: ric_description/komodo/komodo_no_plugins.xacro (robot description, xacro)
@@ -83,5 +83,5 @@
   <joint
     name="komodo_$(arg komodo_id)_FR_Wheel_joint"
-    type="continuous">
+    type="fixed">
     <origin
       xyz="0.173999999999995 -0.2009 0"
@@ -136,5 +136,5 @@
   <joint
     name="komodo_$(arg komodo_id)_FL_Wheel_joint"
-    type="continuous">
+    type="fixed">
     <origin
       xyz="0.173999999999995 0.2009 0"
@@ -189,5 +189,5 @@
   <joint
     name="komodo_$(arg komodo_id)_RR_Wheel_joint"
-    type="continuous">
+    type="fixed">
     <origin
       xyz="-0.156000000000005 -0.2009 0"
@@ -242,5 +242,5 @@
   <joint
     name="komodo_$(arg komodo_id)_RL_Wheel_joint"
-    type="continuous">
+    type="fixed">
     <origin
       xyz="-0.156000000000005 0.2009 0"

File: ric_description/komodo/komodo_no_plugins2.xacro (robot description, xacro)
@@ -1,4 +1,4 @@
 <?xml version="1.0"?>
-<robot xmlns:xacro="http://www.ros.org/wiki/ric" name="komodo">
+<robot xmlns:xacro="http://www.ros.org/wiki/ric" name="ric_description">
   <link
     name="base_link">
@@ -8,33 +8,34 @@
         rpy="0 0 0" />
       <mass
-        value="45.0894999160313" />
-      <inertia
-        ixx="0.723503030508731"
-        ixy="-46.8485359152423E-05"
-        ixz="-0.0875564429068847"
-        iyy="1.38127064231828"
-        iyz="11.9695110167269E-05"
-        izz="1.94371448739423" />
-    </inertial>
-    <visual>
-      <origin
-        xyz="0 0 0"
-        rpy="0 0 0" />
-      <geometry>
-        <mesh
-          filename="package://ric_description/komodo/meshes/col_base_link.STL" />
-      </geometry>
-      <material
-         name="">
-       <color rgba="0.52941176470588 0.52941176470588 0.52941176470588 1" />
-      </material>
-    </visual>
-    <collision>
-      <origin
-        xyz="-0.065 0 0"
-        rpy="0 0 0" />
-      <geometry>
-        <mesh
-          filename="package://ric_description/komodo/meshes/col_base_link.STL" />
+        value="4.50894999160313" />
+      <inertia
+        ixx="0.0723503030508731"
+        ixy="-4.68485359152423E-05"
+        ixz="-0.00875564429068847"
+        iyy="0.138127064231828"
+        iyz="1.19695110167269E-05"
+        izz="0.194371448739423" />
+    </inertial>
+    <visual>
+      <origin
+        xyz="0 0 0"
+        rpy="0 0 0" />
+      <geometry>
+        <mesh
+          filename="package://ric_description/komodo/meshes/base_link.STL" />
+      </geometry>
+      <material
+        name="">
+        <color
+          rgba="0.52941176470588 0.52941176470588 0.52941176470588 1" />
+      </material>
+    </visual>
+    <collision>
+      <origin
+        xyz="0 0 0"
+        rpy="0 0 0" />
+      <geometry>
+        <mesh
+          filename="package://ric_description/komodo/meshes/base_link.STL" />
       </geometry>
     </collision>
@@ -73,10 +74,8 @@
       <origin
         xyz="0 0 0"
-        rpy="0 1.5 0" />
-      <geometry>
-       <!--mesh
-          filename="package://ric_description/komodo/meshes_elevator/FR_Wheel_link.STL" /-->
-        <cylinder length="0.05" radius="0.1"
-          />
+        rpy="0 0 0" />
+      <geometry>
+        <mesh
+          filename="package://ric_description/komodo/meshes/FR_Wheel_link.STL" />
       </geometry>
     </collision>
@@ -87,5 +86,5 @@
     <origin
       xyz="0.173999999999995 -0.2009 0"
-      rpy="2.62229105359916E-15 6.9308460464278E-17 1.5707963267949" />
+      rpy="2.62229105359916E-15 6.9308460464278E-17 -1.5707963267949" />
     <parent
       link="base_link" />
@@ -128,10 +127,8 @@
       <origin
         xyz="0 0 0"
-        rpy="0 1.5 0" />
-      <geometry>
-       <!--mesh
-          filename="package://ric_description/komodo/meshes_elevator/FR_Wheel_link.STL" /-->
-        <cylinder length="0.05" radius="0.1"
-          />
+        rpy="0 0 0" />
+      <geometry>
+        <mesh
+          filename="package://ric_description/komodo/meshes/FL_Wheel_link.STL" />
       </geometry>
     </collision>
@@ -142,5 +139,5 @@
     <origin
       xyz="0.173999999999995 0.2009 0"
-      rpy="-2.62229105359916E-15 6.93084604642783E-17 -1.5707963267949" />
+      rpy="-2.62229105359916E-15 6.93084604642783E-17 1.5707963267949" />
     <parent
       link="base_link" />
@@ -183,10 +180,8 @@
       <origin
         xyz="0 0 0"
-        rpy="0 1.5 0" />
-      <geometry>
-       <!--mesh
-          filename="package://ric_description/komodo/meshes_elevator/FR_Wheel_link.STL" /-->
-        <cylinder length="0.05" radius="0.1"
-          />
+        rpy="0 0 0" />
+      <geometry>
+        <mesh
+          filename="package://ric_description/komodo/meshes/RR_Wheel_link.STL" />
       </geometry>
     </collision>
@@ -197,5 +192,5 @@
     <origin
       xyz="-0.156000000000005 -0.2009 0"
-      rpy="2.62229105359916E-15 -1.59433090848306E-31 1.5707963267949" />
+      rpy="2.62229105359916E-15 -1.59433090848306E-31 -1.5707963267949" />
     <parent
       link="base_link" />
@@ -238,10 +233,8 @@
       <origin
         xyz="0 0 0"
-        rpy="0 1.5 0" />
-      <geometry>
-       <!--mesh
-          filename="package://ric_description/komodo/meshes_elevator/FR_Wheel_link.STL" /-->
-        <cylinder length="0.05" radius="0.1"
-          />
+        rpy="0 0 0" />
+      <geometry>
+        <mesh
+          filename="package://ric_description/komodo/meshes/RL_Wheel_link.STL" />
       </geometry>
     </collision>
@@ -252,5 +245,5 @@
     <origin
       xyz="-0.156000000000005 0.2009 0"
-      rpy="-2.62229105359916E-15 -5.57680208627196E-32 -1.5707963267949" />
+      rpy="-2.62229105359916E-15 -5.57680208627196E-32 1.5707963267949" />
     <parent
       link="base_link" />
@@ -287,5 +280,5 @@
         name="">
         <color
-          rgba="0.752941176470588 0.752941176470588 0.752941176470588 1" />
+          rgba="0.1 0.1 0.1 1" />
       </material>
     </visual>
@@ -340,5 +333,5 @@
         name="">
         <color
-          rgba="0.752941176470588 0.752941176470588 0.752941176470588 1" />
+          rgba="0.1 0.1 0.1 1" />
       </material>
     </visual>
@@ -393,5 +386,5 @@
         name="">
         <color
-          rgba="0.752941176470588 0.752941176470588 0.752941176470588 1" />
+          rgba="0.1 0.1 0.1 1" />
       </material>
     </visual>
@@ -438,5 +431,5 @@
       <origin
         xyz="0 0 0"
-        rpy="-1.57079632649567 1.57079632649567 -1.57079632649567" />
+        rpy="0 0 0" />
       <geometry>
         <mesh
@@ -452,5 +445,5 @@
       <origin
         xyz="0 0 0"
-        rpy="1.57 0 0" />
+        rpy="0 0 0" />
       <geometry>
         <mesh
@@ -464,5 +457,5 @@
     <origin
       xyz="0.262250027816762 0.0875000000000051 0.100000000000001"
-      rpy="0 0 0" />
+      rpy="-1.57079632679489 -6.93084604642783E-17 -1.5707963267949" />
     <parent
       link="base_link" />
@@ -652,8 +645,6 @@
         rpy="0 0 0" />
       <geometry>
-        <!--mesh
-          filename="package://ric_description/komodo/meshes/base_rotation_link.STL" /-->
-	<mesh
-          filename="package://ric_description/komodo/meshes/col_base_rotation_link.STL" />
+        <mesh
+          filename="package://ric_description/komodo/meshes/base_rotation_link.STL" />
       </geometry>
       <material
@@ -669,5 +660,5 @@
       <geometry>
         <mesh
-          filename="package://ric_description/komodo/meshes/col_base_rotation_link.STL" /> <!-- Simplified -->
+          filename="package://ric_description/komodo/meshes/base_rotation_link.STL" />
       </geometry>
     </collision>
@@ -686,7 +677,7 @@
       xyz="0 0 1" />
     <limit
-      lower="-3.14"
-      upper="3.14"
-      effort="10"
+      lower="-1.57079"
+      upper="1.57079"
+      effort="0"
       velocity="0" />
   </joint>
@@ -713,5 +704,5 @@
       <geometry>
         <mesh
-          filename="package://ric_description/komodo/meshes/col_shoulder_link.STL" /> <!-- Simplified -->
+          filename="package://ric_description/komodo/meshes/shoulder_link.STL" />
       </geometry>
       <material
@@ -727,5 +718,5 @@
       <geometry>
         <mesh
-          filename="package://ric_description/komodo/meshes/col_shoulder_link.STL" /> <!-- Simplified -->
+          filename="package://ric_description/komodo/meshes/shoulder_link.STL" />
       </geometry>
     </collision>
@@ -744,7 +735,7 @@
       xyz="0 1 0" />
     <limit
-      lower="-1.57"
-      upper="1.57"
-      effort="2000"
+      lower="-1.692969"
+      upper="1.692969"
+      effort="0"
       velocity="0" />
   </joint>
@@ -771,5 +762,5 @@
       <geometry>
         <mesh
-          filename="package://ric_description/komodo/meshes/col_elbow1_link.STL" />  <!-- Simplified -->
+          filename="package://ric_description/komodo/meshes/elbow1_link.STL" />
       </geometry>
       <material
@@ -785,5 +776,5 @@
       <geometry>
         <mesh
-         filename="package://ric_description/komodo/meshes/col_elbow1_link.STL" />  <!-- Simplified -->
+          filename="package://ric_description/komodo/meshes/elbow1_link.STL" />
       </geometry>
     </collision>
@@ -802,7 +793,7 @@
       xyz="-0.999999999998754 0 0" />
     <limit
-      lower="-3.14"
-      upper="3.14"
-      effort="100"
+      lower="-2.4434"
+      upper="2.4434"
+      effort="0"
       velocity="0" />
   </joint>
@@ -816,5 +807,5 @@
         value="1.12138857800426" />
       <inertia
-        ixx="0.0011156254663426"
+        ixx="0.0110599202589784"
         ixy="3.04261287700186E-07"
         ixz="-1.22468079415109E-06"
@@ -829,5 +820,5 @@
       <geometry>
         <mesh
-           filename="package://ric_description/komodo/meshes/col_elbow2_link.STL" />  <!-- Simplified -->
+          filename="package://ric_description/komodo/meshes/elbow2_link.STL" />
       </geometry>
       <material
@@ -843,5 +834,5 @@
       <geometry>
         <mesh
-          filename="package://ric_description/komodo/meshes/col_elbow2_link.STL" />  <!-- Simplified -->
+          filename="package://ric_description/komodo/meshes/elbow2_link.STL" />
       </geometry>
     </collision>
@@ -852,5 +843,5 @@
     <origin
       xyz="0 0 0.223999999999899"
-      rpy="-4.51048856041191E-16 3.35869632765754E-16 0" />
+      rpy="-4.51048856041191E-16 3.35869632765754E-16 1.57079632687657" />
     <parent
       link="elbow1_link" />
@@ -858,9 +849,9 @@
       link="elbow2_link" />
     <axis
-      xyz="0 1 0" />
+      xyz="1 0 0" />
     <limit
-      lower="-3.14"
-      upper="3.14"
-      effort="10"
+      lower="-2.4434"
+      upper="2.4434"
+      effort="0"
       velocity="0" />
   </joint>
@@ -869,5 +860,5 @@
     <inertial>
       <origin
-        xyz="0 0 0"
+        xyz="-0.000140374211043626 4.00707618562063E-10 0.0303673809619358"
         rpy="0 0 0" />
       <mass
@@ -887,19 +878,19 @@
       <geometry>
         <mesh
-        filename="package://ric_description/komodo/meshes/col_wrist_link.STL" />  <!-- Simplified -->
-      </geometry>
-      <material
-        name="">
-        <color
-          rgba="0.4 0.4 0.4 1" />
-      </material>
-    </visual>
-    <collision>
-      <origin
-        xyz="0 0 0"
-        rpy="0 0 0" />
-      <geometry>
-        <mesh
-          filename="package://ric_description/komodo/meshes/col_wrist_link.STL" />  <!-- Simplified -->
+          filename="package://ric_description/komodo/meshes/wrist_link.STL" />
+      </geometry>
+      <material
+        name="">
+        <color
+          rgba="0.3 0.3 0.3 1" />
+      </material>
+    </visual>
+    <collision>
+      <origin
+        xyz="0 0 0"
+        rpy="0 0 0" />
+      <geometry>
+        <mesh
+          filename="package://ric_description/komodo/meshes/wrist_link.STL" />
       </geometry>
     </collision>
@@ -909,6 +900,6 @@
     type="revolute">
     <origin
-      xyz="0.0137 0 0.244749999999997"
-      rpy="0 0 0" />
+      xyz="0 -0.0130999999999997 0.244749999999997"
+      rpy="-4.43972025628984E-16 -3.35842401421639E-15 -1.57079632687657" />
     <parent
       link="elbow2_link" />
@@ -918,7 +909,7 @@
       xyz="0 0 0.999999999998754" />
     <limit
-      lower="-3.14"
-      upper="3.14"
-      effort="10"
+      lower="-1.91986"
+      upper="1.91986"
+      effort="0"
       velocity="0" />
   </joint>
@@ -932,18 +923,18 @@
         value="0.0111981711598485" />
       <inertia
-        ixx="0.000486392340366094"
-        ixy="4.20757000035677E-12"
-        ixz="-3.91843889020299E-06"
-        iyy="0.000211170064630335"
-        iyz="2.79335159568522E-12"
-        izz="0.000437528795624211" />
-    </inertial>
-    <visual>
-      <origin
-        xyz="0 0 0"
-        rpy="0 0 0" />
-      <geometry>
-        <mesh
-          filename="package://ric_description/komodo/meshes/col_left_finger_link.STL" />  <!-- Simplified -->
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