Commit message: [ric_gazebo]: fix collision

File: ric_description/komodo/komodo_elevator2_for_gazebo.xacro (robot description, xacro)
@@ -74,8 +74,8 @@
       <origin
         xyz="0 0 0"
-        rpy="0 0 0" />
-      <geometry>
-        <mesh
-          filename="package://ric_description/komodo/meshes_elevator/FR_Wheel_link.STL" />
+        rpy="0 1.5 0" />
+      <geometry>
+        <!-- <mesh filename="package://ric_description/komodo/meshes_elevator/FR_Wheel_link.STL" /> -->
+        <cylinder length="0.05" radius="0.1" />
       </geometry>
     </collision>
@@ -127,8 +127,8 @@
       <origin
         xyz="0 0 0"
-        rpy="0 0 0" />
-      <geometry>
-        <mesh
-          filename="package://ric_description/komodo/meshes_elevator/FL_Wheel_link.STL" />
+        rpy="0 1.5 0" />
+      <geometry>
+        <!-- <mesh filename="package://ric_description/komodo/meshes_elevator/FL_Wheel_link.STL" /> -->
+        <cylinder length="0.05" radius="0.1" />
       </geometry>
     </collision>
@@ -180,8 +180,8 @@
       <origin
         xyz="0 0 0"
-        rpy="0 0 0" />
-      <geometry>
-        <mesh
-          filename="package://ric_description/komodo/meshes_elevator/RR_Wheel_link.STL" />
+        rpy="0 1.5 0" />
+      <geometry>
+        <!-- <mesh filename="package://ric_description/komodo/meshes_elevator/RR_Wheel_link.STL" /> -->
+        <cylinder length="0.05" radius="0.1" />
       </geometry>
     </collision>
@@ -233,8 +233,8 @@
       <origin
         xyz="0 0 0"
-        rpy="0 0 0" />
-      <geometry>
-        <mesh
-          filename="package://ric_description/komodo/meshes_elevator/RL_Wheel_link.STL" />
+        rpy="0 1.5 0" />
+      <geometry>
+        <!-- <mesh filename="package://ric_description/komodo/meshes_elevator/RL_Wheel_link.STL" /> -->
+        <cylinder length="0.05" radius="0.1" />
       </geometry>
     </collision>
