Commit message: First Lizi Sim commit - 26.04

File: ric_description/lizi/lizi.xacro (robot description, xacro)
@@ -1,7 +1,7 @@
 <?xml version="1.0"?>
 <robot xmlns:xacro="http://www.ros.org/wiki/lizi_robot" name="lizi_urdf">
-<xacro:property name="lizi_color" value="0 0.517 0.26 1" />
-  <link
-    name="lizi_$(arg lizi_id)_base_link">
+<xacro:property name="lizi_color" value="0.1 0.0 0.1 1" />
+  <link
+    name="base_link">
     <inertial>
       <origin
@@ -43,5 +43,5 @@
   </link>
   <link
-    name="lizi_$(arg lizi_id)_FL_Wheel_link">
+    name="FL_Wheel_link">
     <inertial>
       <origin
@@ -61,5 +61,5 @@
       <origin
         xyz="0 0 0"
-        rpy="0 0 0" />
+        rpy="3.14159265359 0 0" />
       <geometry>
         <mesh
@@ -75,26 +75,28 @@
       <origin
         xyz="0 0 0"
-        rpy="0 0 0" />
-      <geometry>
-        <mesh
-          filename="package://ric_description/lizi/meshes/FL_Wheel_Link.STL" />
-      </geometry>
-    </collision>
-  </link>
-  <joint
-    name="lizi_$(arg lizi_id)_FL_Wheel_Joint"
+        rpy="1.5707963267949 0 0" />
+      <geometry>
+        <!--mesh
+          filename="package://ric_description/lizi/meshes/FL_Wheel_Link.STL" /-->
+        <cylinder length="0.02" radius="0.068"
+          />
+      </geometry>
+    </collision>
+  </link>
+  <joint
+    name="FL_Wheel_Joint"
     type="continuous">
     <origin
       xyz="0.118 0.1338 0.026"
-      rpy="0 0 -1.3371E-16" />
-    <parent
-      link="lizi_$(arg lizi_id)_base_link" />
-    <child
-      link="lizi_$(arg lizi_id)_FL_Wheel_link" />
+      rpy="3.14159265359 0 -1.3371E-16" />
+    <parent
+      link="base_link" />
+    <child
+      link="FL_Wheel_link" />
     <axis
       xyz="0 -1 0" />
   </joint>
   <link
-    name="lizi_$(arg lizi_id)_RL_Wheel_link">
+    name="RL_Wheel_link">
     <inertial>
       <origin
@@ -114,5 +116,5 @@
       <origin
         xyz="0 0 0"
-        rpy="0 0 0" />
+        rpy="3.14159265359 0 0" />
       <geometry>
         <mesh
@@ -128,21 +130,23 @@
       <origin
         xyz="0 0 0"
-        rpy="0 0 0" />
-      <geometry>
-        <mesh
-          filename="package://ric_description/lizi/meshes/RL_Wheel_Link.STL" />
-      </geometry>
-    </collision>
-  </link>
-  <joint
-    name="lizi_$(arg lizi_id)_RL_Wheel_Joint"
+        rpy="1.5707963267949 0 0" />
+      <geometry>
+        <!--mesh
+          filename="package://ric_description/lizi/meshes/RL_Wheel_Link.STL" /-->
+<cylinder length="0.02" radius="0.068"
+          />
+      </geometry>
+    </collision>
+  </link>
+  <joint
+    name="RL_Wheel_Joint"
     type="continuous">
     <origin
       xyz="-0.118 0.1338 0.026"
-      rpy="0 0 -6.6853E-16" />
-    <parent
-      link="lizi_$(arg lizi_id)_base_link" />
-    <child
-      link="lizi_$(arg lizi_id)_RL_Wheel_link" />
+      rpy="3.14159265359 0 -6.6853E-16" />
+    <parent
+      link="base_link" />
+    <child
+      link="RL_Wheel_link" />
     <axis
       xyz="0 -1 0" />
@@ -152,5 +156,5 @@
   </joint>
   <link
-    name="lizi_$(arg lizi_id)_RR_Wheel_link">
+    name="RR_Wheel_link">
     <inertial>
       <origin
@@ -184,13 +188,15 @@
       <origin
         xyz="0 0 0"
-        rpy="0 0 0" />
-      <geometry>
-        <mesh
-          filename="package://ric_description/lizi/meshes/RR_Wheel_Link.STL" />
-      </geometry>
-    </collision>
-  </link>
-  <joint
-    name="lizi_$(arg lizi_id)_RR_Wheel_Joint"
+        rpy="1.5707963267949 0 0" />
+      <geometry>
+        <!--mesh
+          filename="package://ric_description/lizi/meshes/RR_Wheel_Link.STL" /-->
+<cylinder length="0.02" radius="0.068"
+          />
+      </geometry>
+    </collision>
+  </link>
+  <joint
+    name="RR_Wheel_Joint"
     type="continuous">
     <origin
@@ -198,12 +204,12 @@
       rpy="-1.2938E-16 -1.2938E-15 -6.6853E-16" />
     <parent
-      link="lizi_$(arg lizi_id)_base_link" />
-    <child
-      link="lizi_$(arg lizi_id)_RR_Wheel_link" />
+      link="base_link" />
+    <child
+      link="RR_Wheel_link" />
     <axis
       xyz="0 1 0" />
   </joint>
   <link
-    name="lizi_$(arg lizi_id)_FR_Wheel_link">
+    name="FR_Wheel_link">
     <inertial>
       <origin
@@ -237,13 +243,14 @@
       <origin
         xyz="0 0 0"
-        rpy="0 0 0" />
-      <geometry>
-        <mesh
-          filename="package://ric_description/lizi/meshes/FR_Wheel_Link.STL" />
-      </geometry>
-    </collision>
-  </link>
-  <joint
-    name="lizi_$(arg lizi_id)_FR_Wheel_Joint"
+        rpy="1.5707963267949 0 0" />
+      <geometry>
+        <!--mesh
+          filename="package://ric_description/lizi/meshes/FR_Wheel_Link.STL" /-->
+<cylinder length="0.02" radius="0.068"/>
+      </geometry>
+    </collision>
+  </link>
+  <joint
+    name="FR_Wheel_Joint"
     type="continuous">
     <origin
@@ -251,12 +258,12 @@
       rpy="4.4216E-16 -0.0061583 -2.6824E-16" />
     <parent
-      link="lizi_$(arg lizi_id)_base_link" />
-    <child
-      link="lizi_$(arg lizi_id)_FR_Wheel_link" />
+      link="base_link" />
+    <child
+      link="FR_Wheel_link" />
     <axis
       xyz="0 1 0" />
   </joint>
   <link
-    name="lizi_$(arg lizi_id)_Asus_Pan_link">
+    name="Asus_Pan_link">
     <inertial>
       <origin
@@ -298,5 +305,5 @@
   </link>
   <joint
-    name="lizi_$(arg lizi_id)_Asus_Pan_Joint"
+    name="Asus_Pan_Joint"
     type="revolute">
     <origin
@@ -304,7 +311,7 @@
       rpy="2.1253E-16 8.5011E-16 0" />
     <parent
-      link="lizi_$(arg lizi_id)_base_link" />
-    <child
-      link="lizi_$(arg lizi_id)_Asus_Pan_link" />
+      link="base_link" />
+    <child
+      link="Asus_Pan_link" />
     <axis
       xyz="0 0 -1" />
@@ -314,5 +321,5 @@
   </joint>
   <link
-    name="lizi_$(arg lizi_id)_Asus_Camera_link">
+    name="Asus_Camera_link">
     <inertial>
       <origin
@@ -346,5 +353,5 @@
       <origin
         xyz="0 0 0"
-        rpy="0 0 0" />
+        rpy="1.5707963267949 0 0" />
       <geometry>
         <mesh
@@ -354,5 +361,5 @@
   </link>
   <joint
-    name="lizi_$(arg lizi_id)_Asus_Tilt_Joint"
+    name="Asus_Tilt_Joint"
     type="revolute">
     <origin
@@ -360,7 +367,7 @@
       rpy="0 0 0" />
     <parent
-      link="lizi_$(arg lizi_id)_Asus_Pan_link" />
-    <child
-      link="lizi_$(arg lizi_id)_Asus_Camera_link" />
+      link="Asus_Pan_link" />
+    <child
+      link="Asus_Camera_link" />
     <axis
       xyz="0 1 0" />
@@ -370,5 +377,5 @@
   </joint>
   <link
-    name="lizi_$(arg lizi_id)_Right_URF_link">
+    name="Right_URF_link">
     <inertial>
       <origin
@@ -410,5 +417,5 @@
   </link>
   <joint
-    name="lizi_$(arg lizi_id)_Right_URF_Joint"
+    name="Right_URF_Joint"
     type="fixed">
     <origin
@@ -416,12 +423,12 @@
       rpy="0 2.6072E-16 -1.57" />
     <parent
-      link="lizi_$(arg lizi_id)_base_link" />
-    <child
-      link="lizi_$(arg lizi_id)_Right_URF_link" />
+      link="base_link" />
+    <child
+      link="Right_URF_link" />
     <axis
       xyz="0 0 0" />
   </joint>
   <link
-    name="lizi_$(arg lizi_id)_Left_URF_link">
+    name="Left_URF_link">
     <inertial>
       <origin
@@ -463,5 +470,5 @@
   </link>
   <joint
-    name="lizi_$(arg lizi_id)_Left_URF_Joint"
+    name="Left_URF_Joint"
     type="fixed">
     <origin
@@ -469,12 +476,12 @@
       rpy="0 0 1.57" />
     <parent
-      link="lizi_$(arg lizi_id)_base_link" />
-    <child
-      link="lizi_$(arg lizi_id)_Left_URF_link" />
+      link="base_link" />
+    <child
+      link="Left_URF_link" />
     <axis
       xyz="0 0 0" />
   </joint>
   <link
-    name="lizi_$(arg lizi_id)_Rear_URF_link">
+    name="Rear_URF_link">
     <inertial>
       <origin
@@ -516,5 +523,5 @@
   </link>
   <joint
-    name="lizi_$(arg lizi_id)_Rear_URF_Joint"
+    name="Rear_URF_Joint"
     type="fixed">
     <origin
@@ -522,12 +529,12 @@
       rpy="0 0 3.14" />
     <parent
-      link="lizi_$(arg lizi_id)_base_link" />
-    <child
-      link="lizi_$(arg lizi_id)_Rear_URF_link" />
+      link="base_link" />
+    <child
+      link="Rear_URF_link" />
     <axis
       xyz="0 0 0" />
   </joint>
   <link
-    name="lizi_$(arg lizi_id)_Laser_link">
+    name="Laser_link">
     <inertial>
       <origin
@@ -569,5 +576,5 @@
   </link>
   <joint
-    name="lizi_$(arg lizi_id)_Laser_Joint"
+    name="Laser_Joint"
     type="fixed">
     <origin
@@ -575,12 +582,12 @@
       rpy="2.1253E-16 8.5011E-16 -2.6741E-16" />
     <parent
-      link="lizi_$(arg lizi_id)_base_link" />
-    <child
-      link="lizi_$(arg lizi_id)_Laser_link" />
+      link="base_link" />
+    <child
+      link="Laser_link" />
     <axis
       xyz="0 0 0" />
   </joint>
   <link
-    name="lizi_$(arg lizi_id)_Camera_link">
+    name="Camera_link">
     <inertial>
       <origin
@@ -622,5 +629,5 @@
   </link>
   <joint
-    name="lizi_$(arg lizi_id)_Camera_Joint"
+    name="Camera_Joint"
     type="fixed">
     <origin
@@ -628,9 +635,196 @@
       rpy="1.6519E-18 -0.0061583 -2.6824E-16" />
     <parent
-      link="lizi_$(arg lizi_id)_base_link" />
-    <child
-      link="lizi_$(arg lizi_id)_Camera_link" />
+      link="base_link" />
+    <child
+      link="Camera_link" />
     <axis
       xyz="0 0 0" />
   </joint>
+<!-- HW interfaces for ROS CONTROL-->
+  <transmission name="tran1">
+    <type>transmission_interface/SimpleTransmission</type>
+    <joint name="FR_Wheel_Joint">
+<hardwareInterface>EffortJointInterface</hardwareInterface>
+    </joint>
+    <actuator name="motor1">
+      <hardwareInterface>EffortJointInterface</hardwareInterface>
+      <mechanicalReduction>1</mechanicalReduction>
+    </actuator>
+  </transmission>
+  <transmission name="tran2">
+    <type>transmission_interface/SimpleTransmission</type>
+    <joint name="FL_Wheel_Joint">
+<hardwareInterface>EffortJointInterface</hardwareInterface>
+    </joint>
+    <actuator name="motor2">
+      <hardwareInterface>EffortJointInterface</hardwareInterface>
+      <mechanicalReduction>1</mechanicalReduction>
+    </actuator>
+  </transmission>
+  <transmission name="tran3">
+    <type>transmission_interface/SimpleTransmission</type>
+    <joint name="RR_Wheel_Joint">
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
Commit message: Fixed Issues from last E-mail

File: ric_description/lizi/lizi.xacro (robot description, xacro)
@@ -1,5 +1,23 @@
 <?xml version="1.0"?>
 <robot xmlns:xacro="http://www.ros.org/wiki/lizi_robot" name="lizi_urdf">
-<xacro:property name="lizi_color" value="0.1 0.0 0.1 1" />
+<xacro:property name="lizi_color" value="0.0 0.0 0.0 1" />
+<!-- Dummy inertia link & Joint -->
+  <link
+    name="dummy_link">
+</link>
+  <joint
+    name="dummy_joint"
+    type="fixed">
+    <origin
+      xyz="0.0 0.0 0.0"
+      rpy="0 0 0" />
+    <parent
+      link="dummy_link" />
+    <child
+      link="base_link" />
+    <axis
+      xyz="0 0 0" />
+  </joint>
+<!-- Dummy link & node -->
   <link
     name="base_link">
@@ -317,5 +335,7 @@
       xyz="0 0 -1" />
     <limit
-      effort="0"
+      lower="-1"
+      upper="1"
+      effort="10"
       velocity="0" />
   </joint>
@@ -373,5 +393,7 @@
       xyz="0 1 0" />
     <limit
-      effort="0"
+      lower="-1"
+      upper="1"
+      effort="10"
       velocity="0" />
   </joint>
@@ -745,5 +767,5 @@
     <wheelSeparation>0.5</wheelSeparation>
     <wheelDiameter>0.2</wheelDiameter>
-    <robotBaseFrame>base_link</robotBaseFrame>
+    <robotBaseFrame>dummy_link</robotBaseFrame>
     <odometryTopic>odom_$(arg lizi_id)</odometryTopic>
     <odometryFrame>odom_$(arg lizi_id)</odometryFrame>
@@ -828,3 +850,111 @@
     </sensor>
   </gazebo>
+  <!-- Right URF plugin -->
+<gazebo reference="Right_URF_link">
+      <sensor type="ray" name="Right_URF">
+        <pose>0 0 0 0 0 0</pose>
+        <visualize>false</visualize>
+        <ray>
+          <scan>
+            <horizontal>
+              <samples>10</samples>
+              <resolution>1</resolution>
+              <min_angle>-0.5</min_angle>
+              <max_angle> 0.5</max_angle>
+            </horizontal>
+            <vertical>
+              <samples>10</samples>
+              <resolution>1</resolution>
+              <min_angle>-0.2</min_angle>
+              <max_angle> 0.2</max_angle>
+            </vertical>
+          </scan>
+          <range>
+            <min>0.1</min>
+            <max>1.5</max>
+            <resolution>0.01</resolution>
+          </range>
+        </ray>
+        <plugin name="gazebo_ros_Right_URF_controller" filename="libhector_gazebo_ros_sonar.so">
+          <!--gaussianNoise>0.005</gaussianNoise-->
+	  <robotNamespace>/lizi_$(arg lizi_id)</robotNamespace>
+          <topicName>Rangers/Right_URF</topicName>
+          <frameId>/lizi_$(arg lizi_id)/Right_URF_link</frameId>
+        </plugin>
+	  <always_on>true</always_on>
+	  <update_rate>20.0</update_rate>
+      </sensor>
+    </gazebo>
+  <!-- Left URF plugin -->
+<gazebo reference="Left_URF_link">
+      <sensor type="ray" name="Left_URF">
+        <pose>0 0 0 0 0 0</pose>
+        <visualize>false</visualize>
+        <ray>
+          <scan>
+            <horizontal>
+              <samples>10</samples>
+              <resolution>1</resolution>
+              <min_angle>-0.5</min_angle>
+              <max_angle> 0.5</max_angle>
+            </horizontal>
+            <vertical>
+              <samples>10</samples>
+              <resolution>1</resolution>
+              <min_angle>-0.2</min_angle>
+              <max_angle> 0.2</max_angle>
+            </vertical>
+          </scan>
+          <range>
+            <min>0.1</min>
+            <max>1.5</max>
+            <resolution>0.01</resolution>
+          </range>
+        </ray>
+        <plugin name="gazebo_ros_Left_URF_controller" filename="libhector_gazebo_ros_sonar.so">
+          <!--gaussianNoise>0.005</gaussianNoise-->
+	  <robotNamespace>/lizi_$(arg lizi_id)</robotNamespace>
+          <topicName>Rangers/Left_URF</topicName>
+          <frameId>/lizi_$(arg lizi_id)/Left_URF_link</frameId>
+        </plugin>
+	  <always_on>true</always_on>
+	  <update_rate>20.0</update_rate>
+      </sensor>
+    </gazebo>
+  <!-- Rear URF plugin -->
+<gazebo reference="Rear_URF_link">
+      <sensor type="ray" name="Rear_URF">
+        <pose>0 0 0 0 0 0</pose>
+        <visualize>false</visualize>
+        <ray>
+          <scan>
+            <horizontal>
+              <samples>10</samples>
+              <resolution>1</resolution>
+              <min_angle>-0.5</min_angle>
+              <max_angle> 0.5</max_angle>
+            </horizontal>
+            <vertical>
+              <samples>10</samples>
+              <resolution>1</resolution>
+              <min_angle>-0.2</min_angle>
+              <max_angle> 0.2</max_angle>
+            </vertical>
+          </scan>
+          <range>
+            <min>0.1</min>
+            <max>1.5</max>
+            <resolution>0.01</resolution>
+          </range>
+        </ray>
+        <plugin name="gazebo_ros_Rear_URF_controller" filename="libhector_gazebo_ros_sonar.so">
+          <!--gaussianNoise>0.005</gaussianNoise-->
+	  <robotNamespace>/lizi_$(arg lizi_id)</robotNamespace>
+          <topicName>Rangers/Rear_URF</topicName>
+          <frameId>/lizi_$(arg lizi_id)/Rear_URF_link</frameId>
+        </plugin>
+	  <always_on>true</always_on>
+	  <update_rate>20.0</update_rate>
+      </sensor>
+    </gazebo>
 </robot>
