Commit message: gazebo updates

File: ric_description/lizi/lizi.xacro (robot description, xacro)
@@ -814,10 +814,10 @@
     </sensor>
 </gazebo>
-  <!-- hokuyo laser plugin -->
+  <!-- hokuyo URG-04LX laser plugin -->
   <gazebo reference="Laser_link">
     <sensor type="ray" name="head_hokuyo_sensor">
       <pose>0 0 0 0 0 0</pose>
       <visualize>false</visualize>
-      <update_rate>40</update_rate>
+      <update_rate>10</update_rate>
       <ray>
         <scan>
@@ -830,6 +830,6 @@
         </scan>
         <range>
-          <min>0.10</min>
-          <max>30.0</max>
+          <min>0.06</min>
+          <max>4.095</max>
           <resolution>0.01</resolution>
         </range>

File: ric_gazebo/robots/lizi/lizi.xacro (robot description, xacro)
@@ -1,7 +1,7 @@
 <?xml version="1.0"?>
-<robot xmlns:xacro="http://www.ros.org/wiki/lizi_robot" name="$(arg ns)_urdf">
+<robot xmlns:xacro="http://www.ros.org/wiki/lizi_robot" name="lizi_urdf">
 <xacro:property name="lizi_color" value="0.0 0.7 0.0 1" />
 <!-- Dummy inertia link & Joint -->
-   <link
+  <link
     name="dummy_link">
 </link>
@@ -24,25 +24,25 @@
     <inertial>
       <origin
-        xyz="-0.036889 0.00027038 0.069426"
-        rpy="0 0 0" />
-      <mass
-        value="4.706" />
-      <inertia
-        ixx="0.032024"
-        ixy="0.00038846"
-        ixz="-0.0046108"
-        iyy="0.065583"
-        iyz="2.8552E-06"
-        izz="0.076391" />
-    </inertial>
-    <visual>
-      <origin
-        xyz="0 0 0"
-        rpy="0 0 0" />
-      <geometry>
-        <mesh filename="package://ric_description/lizi/meshes/base_link.STL" />
-      </geometry>
-      <material
-        name="">
+	xyz="-0.036889 0.00027038 0.069426"
+	rpy="0 0 0" />
+      <mass
+	value="4.706" />
+      <inertia
+	ixx="0.032024"
+	ixy="0.00038846"
+	ixz="-0.0046108"
+	iyy="0.065583"
+	iyz="2.8552E-06"
+	izz="0.076391" />
+    </inertial>
+    <visual>
+      <origin
+	xyz="0 0 0"
+	rpy="0 0 0" />
+      <geometry>
+	<mesh filename="package://ric_description/lizi/meshes/base_link.STL" />
+      </geometry>
+      <material
+	name="">
 	<color rgba="${lizi_color}" />
       </material>
@@ -50,8 +50,8 @@
     <collision>
       <origin
-        xyz="0 0 0"
-        rpy="0 0 0" />
-      <geometry>
-	   <mesh filename="package://ric_description/lizi/meshes/base_link.STL" />
+	xyz="0 0 0"
+	rpy="0 0 0" />
+      <geometry>
+	  <mesh filename="package://ric_description/lizi/meshes/base_link.STL" />
       </geometry>
     </collision>
@@ -64,43 +64,43 @@
     <inertial>
       <origin
-        xyz="2.9411E-11 -0.0075967 5.8231E-11"
-        rpy="0 0 0" />
-      <mass
-        value="0.4084" />
-      <inertia
-        ixx="0.00059356"
-        ixy="3.4979E-14"
-        ixz="-4.6514E-14"
-        iyy="0.0011268"
-        iyz="5.6928E-14"
-        izz="0.00059356" />
-    </inertial>
-    <visual>
-      <origin
-        xyz="0 0 0"
-        rpy="3.14159265359 0 0" />
-      <geometry>
-        <mesh
-          filename="package://ric_description/lizi/meshes/FL_Wheel_Link.STL" />
-      </geometry>
-      <material
-        name="">
-        <color
-          rgba="0.2 0.2 0.2 1" />
+	xyz="2.9411E-11 -0.0075967 5.8231E-11"
+	rpy="0 0 0" />
+      <mass
+	value="0.4084" />
+      <inertia
+	ixx="0.00059356"
+	ixy="3.4979E-14"
+	ixz="-4.6514E-14"
+	iyy="0.0011268"
+	iyz="5.6928E-14"
+	izz="0.00059356" />
+    </inertial>
+    <visual>
+      <origin
+	xyz="0 0 0"
+	rpy="3.14159265359 0 0" />
+      <geometry>
+	<mesh
+	  filename="package://ric_description/lizi/meshes/FL_Wheel_Link.STL" />
+      </geometry>
+      <material
+	name="">
+	<color
+	  rgba="0.2 0.2 0.2 1" />
       </material>
     </visual>
     <collision>
       <origin
-        xyz="0 0 0"
-        rpy="1.5707963267949 0 0" />
-      <geometry>
-        <!--mesh
-          filename="package://ric_description/lizi/meshes/FL_Wheel_Link.STL" /-->
-        <cylinder length="0.02" radius="0.065"
-          />
-      </geometry>
-    </collision>
-  </link>
-     <gazebo reference="FL_Wheel_link">
+	xyz="0 0 0"
+	rpy="1.5707963267949 0 0" />
+      <geometry>
+	<!--mesh
+	  filename="package://ric_description/lizi/meshes/FL_Wheel_Link.STL" /-->
+	<cylinder length="0.02" radius="0.065"
+	  />
+      </geometry>
+    </collision>
+  </link>
+    <gazebo reference="FL_Wheel_link">
     <material>Gazebo/Grey</material>
 </gazebo>
@@ -122,43 +122,43 @@
     <inertial>
       <origin
-        xyz="2.9411E-11 -0.0035967 5.8231E-11"
-        rpy="0 0 0" />
-      <mass
-        value="0.4084" />
-      <inertia
-        ixx="0.00059356"
-        ixy="3.4979E-14"
-        ixz="-4.6514E-14"
-        iyy="0.0011268"
-        iyz="5.6928E-14"
-        izz="0.00059356" />
-    </inertial>
-    <visual>
-      <origin
-        xyz="0 0 0"
-        rpy="3.14159265359 0 0" />
-      <geometry>
-        <mesh
-          filename="package://ric_description/lizi/meshes/RL_Wheel_Link.STL" />
-      </geometry>
-      <material
-        name="">
-        <color
-          rgba="0.2 0.2 0.2 1" />
+	xyz="2.9411E-11 -0.0035967 5.8231E-11"
+	rpy="0 0 0" />
+      <mass
+	value="0.4084" />
+      <inertia
+	ixx="0.00059356"
+	ixy="3.4979E-14"
+	ixz="-4.6514E-14"
+	iyy="0.0011268"
+	iyz="5.6928E-14"
+	izz="0.00059356" />
+    </inertial>
+    <visual>
+      <origin
+	xyz="0 0 0"
+	rpy="3.14159265359 0 0" />
+      <geometry>
+	<mesh
+	  filename="package://ric_description/lizi/meshes/RL_Wheel_Link.STL" />
+      </geometry>
+      <material
+	name="">
+	<color
+	  rgba="0.2 0.2 0.2 1" />
       </material>
     </visual>
     <collision>
       <origin
-        xyz="0 0 0"
-        rpy="1.5707963267949 0 0" />
-      <geometry>
-        <!--mesh
-          filename="package://ric_description/lizi/meshes/RL_Wheel_Link.STL" /-->
+	xyz="0 0 0"
+	rpy="1.5707963267949 0 0" />
+      <geometry>
+	<!--mesh
+	  filename="package://ric_description/lizi/meshes/RL_Wheel_Link.STL" /-->
 <cylinder length="0.02" radius="0.065"
-          />
-      </geometry>
-    </collision>
-  </link>
-   <gazebo reference="RR_Wheel_link">
+	  />
+      </geometry>
+    </collision>
+  </link>
+  <gazebo reference="RR_Wheel_link">
     <material>Gazebo/Grey</material>
 </gazebo>
@@ -183,43 +183,43 @@
     <inertial>
       <origin
-        xyz="-2.9411E-11 0.0035967 5.8231E-11"
-        rpy="0 0 0" />
-      <mass
-        value="0.4084" />
-      <inertia
-        ixx="0.00059356"
-        ixy="3.4979E-14"
-        ixz="4.6514E-14"
-        iyy="0.0011268"
-        iyz="-5.6928E-14"
-        izz="0.00059356" />
-    </inertial>
-    <visual>
-      <origin
-        xyz="0 0 0"
-        rpy="0 0 0" />
-      <geometry>
-        <mesh
-          filename="package://ric_description/lizi/meshes/RR_Wheel_Link.STL" />
-      </geometry>
-      <material
-        name="">
-        <color
-          rgba="0.2 0.2 0.2 1" />
+	xyz="-2.9411E-11 0.0035967 5.8231E-11"
+	rpy="0 0 0" />
+      <mass
+	value="0.4084" />
+      <inertia
+	ixx="0.00059356"
+	ixy="3.4979E-14"
+	ixz="4.6514E-14"
+	iyy="0.0011268"
+	iyz="-5.6928E-14"
+	izz="0.00059356" />
+    </inertial>
+    <visual>
+      <origin
+	xyz="0 0 0"
+	rpy="0 0 0" />
+      <geometry>
+	<mesh
+	  filename="package://ric_description/lizi/meshes/RR_Wheel_Link.STL" />
+      </geometry>
+      <material
+	name="">
+	<color
+	  rgba="0.2 0.2 0.2 1" />
       </material>
     </visual>
     <collision>
       <origin
-        xyz="0 0 0"
-        rpy="1.5707963267949 0 0" />
-      <geometry>
-        <!--mesh
-          filename="package://ric_description/lizi/meshes/RR_Wheel_Link.STL" /-->
+	xyz="0 0 0"
+	rpy="1.5707963267949 0 0" />
+      <geometry>
+	<!--mesh
+	  filename="package://ric_description/lizi/meshes/RR_Wheel_Link.STL" /-->
 <cylinder length="0.02" radius="0.065"
-          />
-      </geometry>
-    </collision>
-  </link>
-          <gazebo reference="RR_Wheel_link">
+	  />
+      </geometry>
+    </collision>
+  </link>
+	  <gazebo reference="RR_Wheel_link">
     <material>Gazebo/Grey</material>
 </gazebo>
@@ -241,42 +241,42 @@
     <inertial>
       <origin
-        xyz="-2.9052E-11 0.0035967 5.8411E-11"
-        rpy="0 0 0" />
-      <mass
-        value="0.4084" />
-      <inertia
-        ixx="0.00059356"
-        ixy="3.4627E-14"
-        ixz="4.9977E-14"
-        iyy="0.0011268"
-        iyz="-5.7142E-14"
-        izz="0.00059356" />
-    </inertial>
-    <visual>
-      <origin
-        xyz="0 0 0"
-        rpy="0 0 0" />
-      <geometry>
-        <mesh
-          filename="package://ric_description/lizi/meshes/FR_Wheel_Link.STL" />
-      </geometry>
-      <material
-        name="">
-        <color
-          rgba="0.2 0.2 0.2 1" />
+	xyz="-2.9052E-11 0.0035967 5.8411E-11"
+	rpy="0 0 0" />
+      <mass
+	value="0.4084" />
+      <inertia
+	ixx="0.00059356"
+	ixy="3.4627E-14"
+	ixz="4.9977E-14"
+	iyy="0.0011268"
+	iyz="-5.7142E-14"
+	izz="0.00059356" />
+    </inertial>
+    <visual>
+      <origin
+	xyz="0 0 0"
+	rpy="0 0 0" />
+      <geometry>
+	<mesh
+	  filename="package://ric_description/lizi/meshes/FR_Wheel_Link.STL" />
+      </geometry>
+      <material
+	name="">
+	<color
+	  rgba="0.2 0.2 0.2 1" />
       </material>
     </visual>
     <collision>
       <origin
-        xyz="0 0 0"
-        rpy="1.5707963267949 0 0" />
-      <geometry>
-        <!--mesh
-          filename="package://ric_description/lizi/meshes/FR_Wheel_Link.STL" /-->
+	xyz="0 0 0"
+	rpy="1.5707963267949 0 0" />
+      <geometry>
+	<!--mesh
+	  filename="package://ric_description/lizi/meshes/FR_Wheel_Link.STL" /-->
 <cylinder length="0.02" radius="0.065"/>
       </geometry>
     </collision>
   </link>
-        <gazebo reference="FR_Wheel_link">
+	<gazebo reference="FR_Wheel_link">
     <material>Gazebo/Grey</material>
 </gazebo>
@@ -298,37 +298,37 @@
     <inertial>
       <origin
-        xyz="-0.015533 -0.010751 0.019512"
-        rpy="0 0 0" />
-      <mass
-        value="0.016162" />
-      <inertia
-        ixx="5.2781E-06"
-        ixy="1.178E-06"
-        ixz="1.1286E-06"
-        iyy="6.0052E-06"
-        iyz="7.9421E-07"
-        izz="4.7257E-06" />
-    </inertial>
-    <visual>
-      <origin
-        xyz="0 0 0"
-        rpy="0 0 0" />
-      <geometry>
-        <mesh
-          filename="package://ric_description/lizi/meshes/Asus_Pan_Link.STL" />
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