Commit message: gazebo updates

File: ric_gazebo/robots/lizi/lizi.xacro (robot description, xacro)
@@ -1,7 +1,7 @@
 <?xml version="1.0"?>
-<robot xmlns:xacro="http://www.ros.org/wiki/lizi_robot" name="lizi_urdf">
-<xacro:property name="lizi_color" value="0.0 1.0 0.0 1" />
+<robot xmlns:xacro="http://www.ros.org/wiki/lizi_robot" name="$(arg ns)_urdf">
+<xacro:property name="lizi_color" value="0.0 0.7 0.0 1" />
 <!-- Dummy inertia link & Joint -->
-  <link
+   <link
     name="dummy_link">
 </link>
@@ -19,5 +19,5 @@
       xyz="0 0 0" />
   </joint>
-<!-- Dummy link & node -->
+<!--Dummy link & node -->
   <link
     name="base_link">
@@ -41,11 +41,9 @@
         rpy="0 0 0" />
       <geometry>
-        <mesh
-          filename="package://ric_gazebo/robots/lizi/meshes/base_link.STL" />
-      </geometry>
-      <material
-        name="">
-        <color
-          rgba="${lizi_color}" />
+        <mesh filename="package://ric_description/lizi/meshes/base_link.STL" />
+      </geometry>
+      <material
+        name="">
+	<color rgba="${lizi_color}" />
       </material>
     </visual>
@@ -55,9 +53,11 @@
         rpy="0 0 0" />
       <geometry>
-        <mesh
-          filename="package://ric_gazebo/robots/lizi/meshes/base_link.STL" />
-      </geometry>
-    </collision>
-  </link>
+	   <mesh filename="package://ric_description/lizi/meshes/base_link.STL" />
+      </geometry>
+    </collision>
+  </link>
+  <gazebo reference="base_link">
+    <material>Gazebo/$(arg lizi_color_name)</material>
+  </gazebo>
   <link
     name="FL_Wheel_link">
@@ -82,5 +82,5 @@
       <geometry>
         <mesh
-          filename="package://ric_gazebo/robots/lizi/meshes/FL_Wheel_Link.STL" />
+          filename="package://ric_description/lizi/meshes/FL_Wheel_Link.STL" />
       </geometry>
       <material
@@ -96,10 +96,13 @@
       <geometry>
         <!--mesh
-          filename="package://ric_gazebo/robots/lizi/meshes/FL_Wheel_Link.STL" /-->
-        <cylinder length="0.02" radius="0.068"
+          filename="package://ric_description/lizi/meshes/FL_Wheel_Link.STL" /-->
+        <cylinder length="0.02" radius="0.065"
           />
       </geometry>
     </collision>
   </link>
+     <gazebo reference="FL_Wheel_link">
+    <material>Gazebo/Grey</material>
+</gazebo>
   <joint
     name="FL_Wheel_Joint"
@@ -137,5 +140,5 @@
       <geometry>
         <mesh
-          filename="package://ric_gazebo/robots/lizi/meshes/RL_Wheel_Link.STL" />
+          filename="package://ric_description/lizi/meshes/RL_Wheel_Link.STL" />
       </geometry>
       <material
@@ -151,10 +154,13 @@
       <geometry>
         <!--mesh
-          filename="package://ric_gazebo/robots/lizi/meshes/RL_Wheel_Link.STL" /-->
-<cylinder length="0.02" radius="0.068"
+          filename="package://ric_description/lizi/meshes/RL_Wheel_Link.STL" /-->
+<cylinder length="0.02" radius="0.065"
           />
       </geometry>
     </collision>
   </link>
+   <gazebo reference="RR_Wheel_link">
+    <material>Gazebo/Grey</material>
+</gazebo>
   <joint
     name="RL_Wheel_Joint"
@@ -195,5 +201,5 @@
       <geometry>
         <mesh
-          filename="package://ric_gazebo/robots/lizi/meshes/RR_Wheel_Link.STL" />
+          filename="package://ric_description/lizi/meshes/RR_Wheel_Link.STL" />
       </geometry>
       <material
@@ -209,10 +215,13 @@
       <geometry>
         <!--mesh
-          filename="package://ric_gazebo/robots/lizi/meshes/RR_Wheel_Link.STL" /-->
-<cylinder length="0.02" radius="0.068"
+          filename="package://ric_description/lizi/meshes/RR_Wheel_Link.STL" /-->
+<cylinder length="0.02" radius="0.065"
           />
       </geometry>
     </collision>
   </link>
+          <gazebo reference="RR_Wheel_link">
+    <material>Gazebo/Grey</material>
+</gazebo>
   <joint
     name="RR_Wheel_Joint"
@@ -250,5 +259,5 @@
       <geometry>
         <mesh
-          filename="package://ric_gazebo/robots/lizi/meshes/FR_Wheel_Link.STL" />
+          filename="package://ric_description/lizi/meshes/FR_Wheel_Link.STL" />
       </geometry>
       <material
@@ -264,9 +273,12 @@
       <geometry>
         <!--mesh
-          filename="package://ric_gazebo/robots/lizi/meshes/FR_Wheel_Link.STL" /-->
-<cylinder length="0.02" radius="0.068"/>
-      </geometry>
-    </collision>
-  </link>
+          filename="package://ric_description/lizi/meshes/FR_Wheel_Link.STL" /-->
+<cylinder length="0.02" radius="0.065"/>
+      </geometry>
+    </collision>
+  </link>
+        <gazebo reference="FR_Wheel_link">
+    <material>Gazebo/Grey</material>
+</gazebo>
   <joint
     name="FR_Wheel_Joint"
@@ -304,5 +316,5 @@
       <geometry>
         <mesh
-          filename="package://ric_gazebo/robots/lizi/meshes/Asus_Pan_Link.STL" />
+          filename="package://ric_description/lizi/meshes/Asus_Pan_Link.STL" />
       </geometry>
       <material
@@ -318,8 +330,11 @@
       <geometry>
         <mesh
-          filename="package://ric_gazebo/robots/lizi/meshes/Asus_Pan_Link.STL" />
-      </geometry>
-    </collision>
-  </link>
+          filename="package://ric_description/lizi/meshes/Asus_Pan_Link.STL" />
+      </geometry>
+    </collision>
+  </link>
+    <gazebo reference="Asus_Pan_link">
+    <material>Gazebo/Grey</material>
+</gazebo>
   <joint
     name="Asus_Pan_Joint"
@@ -362,5 +377,5 @@
       <geometry>
         <mesh
-          filename="package://ric_gazebo/robots/lizi/meshes/Asus_Camera_Link.STL" />
+          filename="package://ric_description/lizi/meshes/Asus_Camera_Link.STL" />
       </geometry>
       <material
@@ -376,8 +391,11 @@
       <geometry>
         <mesh
-          filename="package://ric_gazebo/robots/lizi/meshes/Asus_Camera_Link.STL" />
-      </geometry>
-    </collision>
-  </link>
+          filename="package://ric_description/lizi/meshes/Asus_Camera_Link.STL" />
+      </geometry>
+    </collision>
+  </link>
+  <gazebo reference="Asus_Camera_link">
+    <material>Gazebo/Grey</material>
+</gazebo>
   <joint
     name="Asus_Tilt_Joint"
@@ -420,5 +438,5 @@
       <geometry>
         <mesh
-          filename="package://ric_gazebo/robots/lizi/meshes/Right_URF_Link.STL" />
+          filename="package://ric_description/lizi/meshes/Right_URF_Link.STL" />
       </geometry>
       <material
@@ -428,11 +446,11 @@
       </material>
     </visual>
-    <collision>
-      <origin
-        xyz="0 0 0"
-        rpy="0 0 0" />
-      <geometry>
-        <mesh
-          filename="package://ric_gazebo/robots/lizi/meshes/Right_URF_Link.STL" />
+   <collision>
+      <origin
+        xyz="0 0 0"
+        rpy="0 0 0" />
+      <geometry>
+        <mesh
+          filename="package://ric_description/lizi/meshes/Right_URF_Link.STL" />
       </geometry>
     </collision>
@@ -473,5 +491,5 @@
       <geometry>
         <mesh
-          filename="package://ric_gazebo/robots/lizi/meshes/Left_URF_Link.STL" />
+          filename="package://ric_description/lizi/meshes/Left_URF_Link.STL" />
       </geometry>
       <material
@@ -487,5 +505,5 @@
       <geometry>
         <mesh
-          filename="package://ric_gazebo/robots/lizi/meshes/Left_URF_Link.STL" />
+          filename="package://ric_description/lizi/meshes/Left_URF_Link.STL" />
       </geometry>
     </collision>
@@ -526,5 +544,5 @@
       <geometry>
         <mesh
-          filename="package://ric_gazebo/robots/lizi/meshes/Rear_URF_Link.STL" />
+          filename="package://ric_description/lizi/meshes/Rear_URF_Link.STL" />
       </geometry>
       <material
@@ -540,5 +558,5 @@
       <geometry>
         <mesh
-          filename="package://ric_gazebo/robots/lizi/meshes/Rear_URF_Link.STL" />
+          filename="package://ric_description/lizi/meshes/Rear_URF_Link.STL" />
       </geometry>
     </collision>
@@ -579,5 +597,5 @@
       <geometry>
         <mesh
-          filename="package://ric_gazebo/robots/lizi/meshes/Laser_Link.STL" />
+          filename="package://ric_description/lizi/meshes/Laser_Link.STL" />
       </geometry>
       <material
@@ -593,8 +611,11 @@
       <geometry>
         <mesh
-          filename="package://ric_gazebo/robots/lizi/meshes/Laser_Link.STL" />
-      </geometry>
-    </collision>
-  </link>
+          filename="package://ric_description/lizi/meshes/Laser_Link.STL" />
+      </geometry>
+    </collision>
+  </link>
+    <gazebo reference="Laser_link">
+    <material>Gazebo/Grey</material>
+</gazebo>
   <joint
     name="Laser_Joint"
@@ -632,5 +653,5 @@
       <geometry>
         <mesh
-          filename="package://ric_gazebo/robots/lizi/meshes/Camera_Link.STL" />
+          filename="package://ric_description/lizi/meshes/Camera_Link.STL" />
       </geometry>
       <material
@@ -646,8 +667,11 @@
       <geometry>
         <mesh
-          filename="package://ric_gazebo/robots/lizi/meshes/Camera_Link.STL" />
-      </geometry>
-    </collision>
-  </link>
+          filename="package://ric_description/lizi/meshes/Camera_Link.STL" />
+      </geometry>
+    </collision>
+  </link>
+    <gazebo reference="Camera_link">
+    <material>Gazebo/Grey</material>
+</gazebo>
   <joint
     name="Camera_Joint"
@@ -726,5 +750,5 @@
 <gazebo>
   <plugin name="gazebo_ros_control" filename="libgazebo_ros_control.so">
-    <!-- <robotNamespace>/lizi_$(arg lizi_id)</robotNamespace> -->
+    <robotNamespace>$(arg ns)</robotNamespace>
   </plugin>
 </gazebo>
@@ -759,5 +783,5 @@
     <always_on>1</always_on>
     <updateRate>100.0</updateRate>
-    <!--  <robotNamespace>/lizi_$(arg lizi_id)</robotNamespace> -->
+    <robotNamespace>$(arg ns)</robotNamespace>
     <broadcastTF>1</broadcastTF>
     <leftFrontJoint>FL_Wheel_Joint</leftFrontJoint>
@@ -774,5 +798,5 @@
   </plugin>
     <plugin name="gazebo_ros_control" filename="libgazebo_ros_control.so">
-      <!-- <robotNamespace>/lizi_st_$(arg lizi_id)</robotNamespace> -->
+       <robotNamespace>$(arg ns)</robotNamespace>
     </plugin>
 </gazebo>
@@ -796,5 +820,5 @@
       <plugin name="camera_controller" filename="libgazebo_ros_camera.so">
         <alwaysOn>true</alwaysOn>
-	<!--  <robotNamespace>komodo_$(arg komodo_id)</robotNamespace> -->
+	 <robotNamespace>$(arg ns)</robotNamespace>
         <cameraName>Front_Camera</cameraName>
         <imageTopicName>image_raw</imageTopicName>
@@ -838,5 +862,5 @@
 	<pointCloudTopicName>depth/bad_points</pointCloudTopicName>
 	<pointCloudCutoff>0.4</pointCloudCutoff>
-	<pointCloudCutoffMax>4.4</pointCloudCutoffMax>
+        <pointCloudCutoffMax>50.0</pointCloudCutoffMax>
 	<frameName>Asus_Camera_link</frameName>
 	<distortion_k1>0.0</distortion_k1>
@@ -912,5 +936,5 @@
         <plugin name="gazebo_ros_Right_URF_controller" filename="libhector_gazebo_ros_sonar.so">
           <!--gaussianNoise>0.005</gaussianNoise-->
-	  <!-- <robotNamespace>/lizi_$(arg lizi_id)</robotNamespace> -->
+	 <robotNamespace>$(arg ns)</robotNamespace>
           <topicName>Rangers/Right_URF</topicName>
           <frameId>Right_URF_link</frameId>
@@ -948,5 +972,5 @@
         <plugin name="gazebo_ros_Left_URF_controller" filename="libhector_gazebo_ros_sonar.so">
           <!--gaussianNoise>0.005</gaussianNoise-->
-	  <!--  <robotNamespace>/lizi_$(arg lizi_id)</robotNamespace> -->
+	  <robotNamespace>$(arg ns)</robotNamespace>
           <topicName>Rangers/Left_URF</topicName>
           <frameId>Left_URF_link</frameId>
@@ -984,5 +1008,5 @@
         <plugin name="gazebo_ros_Rear_URF_controller" filename="libhector_gazebo_ros_sonar.so">
           <!--gaussianNoise>0.005</gaussianNoise-->
-	  <!--  <robotNamespace>/lizi_$(arg lizi_id)</robotNamespace> -->
+	 <robotNamespace>$(arg ns)</robotNamespace>
           <topicName>Rangers/Rear_URF</topicName>
           <frameId>Rear_URF_link</frameId>

Commit message: lizi gazebo configs

File: ric_gazebo/robots/lizi/lizi.xacro (robot description, xacro)
@@ -1,8 +1,17 @@
 <?xml version="1.0"?>
 <robot xmlns:xacro="http://www.ros.org/wiki/ric_gazebo" name="lizi">
-<xacro:property name="lizi_color" value="0.0 0.7 0.0 1" />
+<xacro:include filename="$(find ric_gazebo)/robots/materials.xacro" />
+<xacro:arg name="ns" default="lizi"/>
+<xacro:arg name="color" default="Green"/>
+<xacro:arg name="gazebo" default="false"/>
+<xacro:arg name="front_camera" default="false"/>
+<xacro:arg name="depth_camera" default="false"/>
+<xacro:arg name="laser_scanner" default="false"/>
+<xacro:arg name="urf" default="false"/>
+<xacro:arg name="imu" default="false"/>
+<xacro:arg name="pan_tilt" default="true"/>
+<xacro:if value="$(arg gazebo)">
 <!-- Dummy inertia link & Joint -->
-  <link
-    name="dummy_link">
+  <link name="dummy_link">
 </link>
   <joint
@@ -19,5 +28,5 @@
       xyz="0 0 0" />
   </joint>
-<!--Dummy link & node -->
+</xacro:if>
   <link
     name="base_link">
@@ -43,8 +52,7 @@
 	<mesh filename="package://ric_description/lizi/meshes/base_link.STL" />
       </geometry>
-      <material
-	name="">
-	<color rgba="${lizi_color}" />
-      </material>
+    <material
+	name="$(arg color)">
+    </material>
     </visual>
     <collision>
@@ -57,7 +65,4 @@
     </collision>
   </link>
-  <gazebo reference="base_link">
-    <material>Gazebo/$(arg lizi_color_name)</material>
-  </gazebo>
   <link
     name="FL_Wheel_link">
@@ -102,7 +107,4 @@
     </collision>
   </link>
-    <gazebo reference="FL_Wheel_link">
-    <material>Gazebo/Grey</material>
-</gazebo>
   <joint
     name="FL_Wheel_Joint"
@@ -160,7 +162,4 @@
     </collision>
   </link>
-  <gazebo reference="RR_Wheel_link">
-    <material>Gazebo/Grey</material>
-</gazebo>
   <joint
     name="RL_Wheel_Joint"
@@ -221,7 +220,4 @@
     </collision>
   </link>
-	  <gazebo reference="RR_Wheel_link">
-    <material>Gazebo/Grey</material>
-</gazebo>
   <joint
     name="RR_Wheel_Joint"
@@ -278,7 +274,4 @@
     </collision>
   </link>
-	<gazebo reference="FR_Wheel_link">
-    <material>Gazebo/Grey</material>
-</gazebo>
   <joint
     name="FR_Wheel_Joint"
@@ -334,7 +327,5 @@
     </collision>
   </link>
-    <gazebo reference="Asus_Pan_link">
-    <material>Gazebo/Grey</material>
-</gazebo>
+<xacro:if value="$(arg pan_tilt)">
   <joint
     name="Asus_Pan_Joint"
@@ -355,4 +346,25 @@
       velocity="0" />
   </joint>
+</xacro:if>
+<xacro:unless value="$(arg pan_tilt)">
+ <joint
+    name="Asus_Pan_Joint"
+    type="fixed">
+    <origin
+      xyz="0.081249 0 0.092091"
+      rpy="2.1253E-16 8.5011E-16 0" />
+    <parent
+      link="base_link" />
+    <child
+      link="Asus_Pan_link" />
+    <axis
+      xyz="0 0 -1" />
+    <limit
+      lower="-1"
+      upper="1"
+      effort="10"
+      velocity="0" />
+  </joint>
+</xacro:unless>
   <link
     name="Asus_Camera_link">
@@ -395,7 +407,5 @@
     </collision>
   </link>
-  <gazebo reference="Asus_Camera_link">
-    <material>Gazebo/Grey</material>
-</gazebo>
+<xacro:if value="$(arg pan_tilt)">
   <joint
     name="Asus_Tilt_Joint"
@@ -416,4 +426,25 @@
       velocity="0" />
   </joint>
+</xacro:if>
+<xacro:unless value="$(arg pan_tilt)">
+  <joint
+    name="Asus_Tilt_Joint"
+    type="fixed">
+    <origin
+      xyz="-0.0004889 -0.00041349 0.08"
+      rpy="0 0 0" />
+    <parent
+      link="Asus_Pan_link" />
+    <child
+      link="Asus_Camera_link" />
+    <axis
+      xyz="0 1 0" />
+    <limit
+      lower="-1"
+      upper="1"
+      effort="10"
+      velocity="0" />
+  </joint>
+  </xacro:unless>
   <link
     name="Right_URF_link">
@@ -456,7 +487,4 @@
     </collision>
   </link>
-<gazebo reference="Right_URF_link">
-    <material>Gazebo/Grey</material>
-</gazebo>
   <joint
     name="Right_URF_Joint"
@@ -512,7 +540,4 @@
     </collision>
   </link>
-  <gazebo reference="Left_URF_link">
-    <material>Gazebo/Grey</material>
-</gazebo>
   <joint
     name="Left_URF_Joint"
@@ -568,7 +593,4 @@
     </collision>
   </link>
-    <gazebo reference="Rear_URF_link">
-    <material>Gazebo/Grey</material>
-</gazebo>
   <joint
     name="Rear_URF_Joint"
@@ -624,7 +646,4 @@
     </collision>
   </link>
-    <gazebo reference="Laser_link">
-    <material>Gazebo/Grey</material>
-</gazebo>
   <joint
     name="Laser_Joint"
@@ -680,7 +699,4 @@
     </collision>
   </link>
-    <gazebo reference="Camera_link">
-    <material>Gazebo/Grey</material>
-</gazebo>
   <joint
     name="Camera_Joint"
@@ -696,4 +712,41 @@
       xyz="0 0 0" />
   </joint>
+  <xacro:if value="$(arg gazebo)">
+      <gazebo reference="base_link">
+    <material>Gazebo/$(arg color)</material>
+  </gazebo>
+    <gazebo reference="FL_Wheel_link">
+    <material>Gazebo/Grey</material>
+</gazebo>
+  <gazebo reference="RR_Wheel_link">
+    <material>Gazebo/Grey</material>
+</gazebo>
+	  <gazebo reference="RR_Wheel_link">
+    <material>Gazebo/Grey</material>
+</gazebo>
+	<gazebo reference="FR_Wheel_link">
+    <material>Gazebo/Grey</material>
+</gazebo>
+    <gazebo reference="Asus_Pan_link">
+    <material>Gazebo/Grey</material>
+</gazebo>
+  <gazebo reference="Asus_Camera_link">
+    <material>Gazebo/Grey</material>
+</gazebo>
+<gazebo reference="Right_URF_link">
+    <material>Gazebo/Grey</material>
+</gazebo>
+  <gazebo reference="Left_URF_link">
+    <material>Gazebo/Grey</material>
+</gazebo>
+    <gazebo reference="Rear_URF_link">
+    <material>Gazebo/Grey</material>
+</gazebo>
+    <gazebo reference="Laser_link">
+    <material>Gazebo/Grey</material>
+</gazebo>
+    <gazebo reference="Camera_link">
+    <material>Gazebo/Grey</material>
+</gazebo>
 <!-- HW interfaces for ROS CONTROL-->
   <transmission name="tran1">
@@ -737,4 +790,5 @@
     </actuator>
   </transmission>
+  <xacro:if value="$(arg pan_tilt)">
   <transmission name="tran5">
     <type>transmission_interface/SimpleTransmission</type>
@@ -757,4 +811,5 @@
     </actuator>
   </transmission>
+  </xacro:if>
 <gazebo>
   <plugin name="gazebo_ros_control" filename="libgazebo_ros_control.so">
@@ -813,4 +868,6 @@
   -->
 </gazebo>
+</xacro:if>
+  <xacro:if value="$(arg front_camera)">
 <!-- front camera -->
   <gazebo reference="Camera_link">
@@ -846,4 +903,6 @@
     </sensor>
   </gazebo>
+</xacro:if>
+  <xacro:if value="$(arg depth_camera)">
   <!-- Asus camera plugin -->
 <gazebo reference="Asus_Camera_link">
@@ -884,4 +943,6 @@
     </sensor>
 </gazebo>
+</xacro:if>
+  <xacro:if value="$(arg laser_scanner)">
   <!-- hokuyo laser plugin -->
   <gazebo reference="Laser_link">
@@ -893,5 +954,5 @@
 	<scan>
 	  <horizontal>
-	    <samples>150</samples>
+	    <samples>200</samples>
 	    <resolution>1.0</resolution>
 	    <min_angle>-1.570796</min_angle>
@@ -920,4 +981,6 @@
     </sensor>
   </gazebo>
+  </xacro:if>
+    <xacro:if value="$(arg urf)">
   <!-- Right URF plugin -->
 <gazebo reference="Right_URF_link">
@@ -1028,4 +1091,6 @@
       </sensor>
     </gazebo>
+    </xacro:if>
+      <xacro:if value="$(arg imu)">
     <!-- IMU -->
   <gazebo>
@@ -1045,3 +1110,4 @@
     </plugin>
 </gazebo>
+</xacro:if>
 </robot>
