Commit message: komodo gazebo updates

File: ric_gazebo/robots/komodo/komodo.xacro (robot description, xacro)
@@ -1,4 +1,15 @@
 <?xml version="1.0"?>
 <robot xmlns:xacro="http://www.ros.org/wiki/ric_gazebo" name="komodo">
+<xacro:include filename="$(find ric_gazebo)/robots/materials.xacro" />
+<xacro:arg name="ns" default="komodo"/>
+<xacro:arg name="color" default="Grey"/>
+<xacro:arg name="gazebo" default="false"/>
+<xacro:arg name="arm_camera" default="false"/>
+<xacro:arg name="front_camera" default="false"/>
+<xacro:arg name="depth_camera" default="false"/>
+<xacro:arg name="laser_scanner" default="false"/>
+<xacro:arg name="urf" default="false"/>
+<xacro:arg name="imu" default="false"/>
+<xacro:if value="$(arg gazebo)">
 <!-- Dummy inertia link & Joint -->
   <link
@@ -18,5 +29,5 @@
       xyz="0 0 0" />
   </joint>
-<!-- Dummy link & node -->
+</xacro:if>
   <link
     name="base_link">
@@ -44,7 +55,6 @@
       </geometry>
       <material
-        name="">
-        <color
-          rgba="0.52941176470588 0.52941176470588 0.52941176470588 1" />
+         name="$(arg color)">
+     <!--  <color rgba="0.52941176470588 0.52941176470588 0.52941176470588 1" /> -->
       </material>
     </visual>
@@ -1164,4 +1174,5 @@
       xyz="1 0 0" />
   </joint>
+    <xacro:if value="$(arg gazebo)">
    <!-- ros_control plugin -->
 <gazebo>
@@ -1322,5 +1333,5 @@
 </gazebo>
   <gazebo reference="base_link">
-    <material>Gazebo/$(arg color_name)</material>
+    <material>Gazebo/$(arg color)</material>
     <mu1>1</mu1>
     <mu2>1</mu2>
@@ -1328,8 +1339,8 @@
   </gazebo>
     <gazebo reference="Arm_base_link">
-    <material>Gazebo/$(arg color_name)</material>
+    <material>Gazebo/$(arg color)</material>
   </gazebo>
       <gazebo reference="sensors_unit_link">
-    <material>Gazebo/$(arg color_name)</material>
+    <material>Gazebo/$(arg color)</material>
   </gazebo>
 <gazebo reference="FR_Wheel_link">
@@ -1360,4 +1371,31 @@
   <material>Gazebo/Grey</material>
 </gazebo>
+<!-- Diff drive -->
+<gazebo>
+  <plugin name="skid_steer_drive_controller" filename="libgazebo_ros_skid_steer_drive.so">
+    <always_on>1</always_on>
+    <updateRate>50.0</updateRate>
+   <robotNamespace>/$(arg ns)</robotNamespace>
+    <broadcastTF>1</broadcastTF>
+    <leftFrontJoint>FL_Wheel_joint</leftFrontJoint>
+    <rightFrontJoint>FR_Wheel_joint</rightFrontJoint>
+    <leftRearJoint>RL_Wheel_joint</leftRearJoint>
+    <rightRearJoint>RR_Wheel_joint</rightRearJoint>
+    <wheelSeparation>0.5</wheelSeparation>
+    <wheelDiameter>0.2</wheelDiameter>
+    <robotBaseFrame>dummy_link</robotBaseFrame>
+    <odometryTopic>diff_driver/odometry</odometryTopic>
+    <odometryFrame>odom_link</odometryFrame>
+    <torque>20</torque>
+    <commandTopic>diff_driver/command</commandTopic>
+  </plugin>
+  <!--
+    <plugin name="gazebo_ros_control" filename="libgazebo_ros_control.so">
+    <robotNamespace>/komodo_st_$(arg komodo_id)</robotNamespace>
+    </plugin>
+  -->
+</gazebo>
+  </xacro:if>
+  <xacro:if value="$(arg arm_camera)">
 <!-- arm camera -->
   <gazebo reference="Arm_Camera_link">
@@ -1393,4 +1431,6 @@
     </sensor>
   </gazebo>
+</xacro:if>
+ <xacro:if value="$(arg front_camera)">
 <!-- front camera -->
   <gazebo reference="Front_Camera_link">
@@ -1426,4 +1466,6 @@
     </sensor>
   </gazebo>
+</xacro:if>
+  <xacro:if value="$(arg depth_camera)">
 <!-- Asus camera  - Gazebo -->
 <gazebo reference="Asus_Camera_link">
@@ -1464,4 +1506,6 @@
     </sensor>
 </gazebo>
+  </xacro:if>
+    <xacro:if value="$(arg laser_scanner)">
   <!-- hokuyo -->
   <gazebo reference="Laser_link">
@@ -1500,4 +1544,6 @@
     </sensor>
   </gazebo>
+  </xacro:if>
+    <xacro:if value="$(arg urf)">
 <!-- SOnar Right URF -->
 <!-- name = komodo_Right_URF
@@ -1512,6 +1558,6 @@
               <samples>10</samples>
               <resolution>1</resolution>
-              <min_angle>-0.5</min_angle>
-              <max_angle> 0.5</max_angle>
+              <min_angle>-0.2</min_angle>
+              <max_angle> 0.2</max_angle>
             </horizontal>
             <vertical>
@@ -1523,6 +1569,6 @@
           </scan>
           <range>
-            <min>0.1</min>
-            <max>1.5</max>
+            <min>0.01</min>
+            <max>5.0</max>
             <resolution>0.01</resolution>
           </range>
@@ -1552,6 +1598,6 @@
               <samples>10</samples>
               <resolution>1</resolution>
-              <min_angle>-0.5</min_angle>
-              <max_angle> 0.5</max_angle>
+              <min_angle>-0.2</min_angle>
+              <max_angle> 0.2</max_angle>
             </horizontal>
             <vertical>
@@ -1563,6 +1609,6 @@
           </scan>
           <range>
-            <min>0.1</min>
-            <max>1.5</max>
+            <min>0.01</min>
+            <max>5.0</max>
             <resolution>0.01</resolution>
           </range>
@@ -1588,6 +1634,6 @@
               <samples>10</samples>
               <resolution>1</resolution>
-              <min_angle>-0.5</min_angle>
-              <max_angle> 0.5</max_angle>
+              <min_angle>-0.2</min_angle>
+              <max_angle> 0.2</max_angle>
             </horizontal>
             <vertical>
@@ -1599,6 +1645,6 @@
           </scan>
           <range>
-            <min>0.1</min>
-            <max>1.5</max>
+            <min>0.01</min>
+            <max>5.0</max>
             <resolution>0.01</resolution>
           </range>
@@ -1612,4 +1658,6 @@
       </sensor>
     </gazebo>
+      </xacro:if>
+ <xacro:if value="$(arg imu)">
 <!-- IMU -->
   <gazebo>
@@ -1627,28 +1675,4 @@
     </plugin>
 </gazebo>
-<!-- Diff drive -->
-<gazebo>
-  <plugin name="skid_steer_drive_controller" filename="libgazebo_ros_skid_steer_drive.so">
-    <always_on>1</always_on>
-    <updateRate>50.0</updateRate>
-   <robotNamespace>/$(arg ns)</robotNamespace>
-    <broadcastTF>1</broadcastTF>
-    <leftFrontJoint>FL_Wheel_joint</leftFrontJoint>
-    <rightFrontJoint>FR_Wheel_joint</rightFrontJoint>
-    <leftRearJoint>RL_Wheel_joint</leftRearJoint>
-    <rightRearJoint>RR_Wheel_joint</rightRearJoint>
-    <wheelSeparation>0.5</wheelSeparation>
-    <wheelDiameter>0.2</wheelDiameter>
-    <robotBaseFrame>dummy_link</robotBaseFrame>
-    <odometryTopic>diff_driver/odometry</odometryTopic>
-    <odometryFrame>odom_link</odometryFrame>
-    <torque>20</torque>
-    <commandTopic>diff_driver/command</commandTopic>
-  </plugin>
-  <!--
-    <plugin name="gazebo_ros_control" filename="libgazebo_ros_control.so">
-    <robotNamespace>/komodo_st_$(arg komodo_id)</robotNamespace>
-    </plugin>
-  -->
-</gazebo>
+</xacro:if>
 </robot>

Commit message: [update]: add condition to the imu component, fusion hz can`t be smaller then pubblish hz

File: ric_gazebo/robots/komodo/komodo.xacro (robot description, xacro)
@@ -13,33 +13,18 @@
 <xacro:if value="$(arg gazebo)">
 <!-- Dummy inertia link & Joint -->
-  <link
-    name="dummy_link">
-</link>
-  <joint
-    name="dummy_joint"
-    type="fixed">
-    <origin
-      xyz="0.0 0.0 0.0"
-      rpy="0 0 0" />
-    <parent
-      link="dummy_link" />
-    <child
-      link="base_link" />
-    <axis
-      xyz="0 0 0" />
+  <link name="dummy_link">
+  </link>
+  <joint name="dummy_joint" type="fixed">
+    <origin xyz="0.0 0.0 0.0" rpy="0 0 0" />
+    <parent link="dummy_link" />
+    <child link="base_link" />
+    <axis xyz="0 0 0" />
   </joint>
 </xacro:if>
-  <link
-    name="base_link">
-    <inertial>
-      <origin
-        xyz="-0.0205330571995271 4.54409684683429E-05 0.00735986203300292"
-        rpy="0 0 0" />
-      <mass
-        value="45.0894999160313" />
-      <inertia
-        ixx="0.723503030508731"
-        ixy="-46.8485359152423E-05"
-        ixz="-0.0875564429068847"
+  <link name="base_link">
+    <inertial>
+      <origin xyz="-0.0205330571995271 4.54409684683429E-05 0.00735986203300292" rpy="0 0 0" />
+      <mass value="45.0894999160313" />
+      <inertia ixx="0.723503030508731" ixy="-46.8485359152423E-05" ixz="-0.0875564429068847"
         iyy="1.38127064231828"
         iyz="11.9695110167269E-05"

Commit message: [update]: ric_gazebo,separate the komodo.xacro in to two files

File: ric_gazebo/robots/komodo/komodo.xacro (robot description, xacro)
@@ -1,1663 +1,526 @@
 <?xml version="1.0"?>
 <robot xmlns:xacro="http://www.ros.org/wiki/ric_gazebo" name="komodo">
-<xacro:include filename="$(find ric_gazebo)/robots/materials.xacro" />
-<xacro:arg name="ns" default="komodo"/>
-<xacro:arg name="color" default="Grey"/>
-<xacro:arg name="gazebo" default="false"/>
-<xacro:arg name="arm_camera" default="false"/>
-<xacro:arg name="front_camera" default="false"/>
-<xacro:arg name="depth_camera" default="false"/>
-<xacro:arg name="laser_scanner" default="false"/>
-<xacro:arg name="urf" default="false"/>
-<xacro:arg name="imu" default="false"/>
-<xacro:if value="$(arg gazebo)">
-<!-- Dummy inertia link & Joint -->
-  <link name="dummy_link">
-  </link>
-  <joint name="dummy_joint" type="fixed">
-    <origin xyz="0.0 0.0 0.0" rpy="0 0 0" />
-    <parent link="dummy_link" />
-    <child link="base_link" />
-    <axis xyz="0 0 0" />
-  </joint>
-</xacro:if>
-  <link name="base_link">
-    <inertial>
-      <origin xyz="-0.0205330571995271 4.54409684683429E-05 0.00735986203300292" rpy="0 0 0" />
-      <mass value="45.0894999160313" />
-      <inertia ixx="0.723503030508731" ixy="-46.8485359152423E-05" ixz="-0.0875564429068847"
-        iyy="1.38127064231828"
-        iyz="11.9695110167269E-05"
-        izz="1.94371448739423" />
-    </inertial>
-    <visual>
-      <origin
-        xyz="0 0 0"
-        rpy="0 0 0" />
-      <geometry>
-        <mesh
-          filename="package://ric_description/komodo/meshes/col_base_link.STL" />
-      </geometry>
-      <material
-         name="$(arg color)">
-     <!--  <color rgba="0.52941176470588 0.52941176470588 0.52941176470588 1" /> -->
-      </material>
-    </visual>
-    <collision>
-      <origin
-        xyz="-0.065 0 0"
-        rpy="0 0 0" />
-      <geometry>
-        <mesh
-          filename="package://ric_description/komodo/meshes/col_base_link.STL" />
-      </geometry>
-    </collision>
-  </link>
-  <link
-    name="FR_Wheel_link">
-    <inertial>
-      <origin
-        xyz="-0.00160662478940524 -2.59227836232889E-06 1.49952129885679E-05"
-        rpy="0 0 0" />
-      <mass
-        value="3.8342752339456" />
-      <inertia
-        ixx="0.0296525526023316"
-        ixy="1.51001308635369E-06"
-        ixz="2.3576732629264E-06"
-        iyy="0.0163749526634419"
-        iyz="1.22545882852199E-06"
-        izz="0.0163720506902763" />
-    </inertial>
-    <visual>
-      <origin
-        xyz="0 0 0"
-        rpy="0 0 0" />
-      <geometry>
-        <mesh
-          filename="package://ric_description/komodo/meshes/FR_Wheel_link.STL" />
-      </geometry>
-      <material
-        name="">
-        <color
-          rgba="0.15 0.15 0.15 1" />
-      </material>
-    </visual>
-    <collision>
-      <origin
-        xyz="0 0 0"
-        rpy="0 1.5 0" />
-      <geometry>
-       <!--mesh
-          filename="package://ric_description/komodo/meshes_elevator/FR_Wheel_link.STL" /-->
-        <cylinder length="0.05" radius="0.1"
-          />
-      </geometry>
-    </collision>
-  </link>
-  <joint
-    name="FR_Wheel_joint"
-    type="continuous">
-    <origin
-      xyz="0.173999999999995 -0.2009 0"
-      rpy="2.62229105359916E-15 6.9308460464278E-17 1.5707963267949" />
-    <parent
-      link="base_link" />
-    <child
-      link="FR_Wheel_link" />
-    <axis
-      xyz="1 0 0" />
-  </joint>
-  <link
-    name="FL_Wheel_link">
-    <inertial>
-      <origin
-        xyz="-0.00160662480262744 -2.59228543311729E-06 1.49951351856364E-05"
-        rpy="0 0 0" />
-      <mass
-        value="3.83427523136739" />
-      <inertia
-        ixx="0.0296525525807749"
-        ixy="1.51001277133356E-06"
-        ixz="2.35766660656153E-06"
-        iyy="0.0163749526386264"
-        iyz="1.2254511654214E-06"
-        izz="0.0163720506916083" />
-    </inertial>
-    <visual>
-      <origin
-        xyz="0 0 0"
-        rpy="0 0 0" />
-      <geometry>
-        <mesh
-          filename="package://ric_description/komodo/meshes/FL_Wheel_link.STL" />
-      </geometry>
-      <material
-        name="">
-        <color
-          rgba="0.15 0.15 0.15 1" />
-      </material>
-    </visual>
-    <collision>
-      <origin
-        xyz="0 0 0"
-        rpy="0 1.5 0" />
-      <geometry>
-       <!--mesh
-          filename="package://ric_description/komodo/meshes_elevator/FR_Wheel_link.STL" /-->
-        <cylinder length="0.05" radius="0.1"
-          />
-      </geometry>
-    </collision>
-  </link>
-  <joint
-    name="FL_Wheel_joint"
-    type="continuous">
-    <origin
-      xyz="0.173999999999995 0.2009 0"
-      rpy="-2.62229105359916E-15 6.93084604642783E-17 -1.5707963267949" />
-    <parent
-      link="base_link" />
-    <child
-      link="FL_Wheel_link" />
-    <axis
-      xyz="-1 0 0" />
-  </joint>
-  <link
-    name="RR_Wheel_link">
-    <inertial>
-      <origin
-        xyz="-0.00160662476834383 -2.59238516814309E-06 1.49950507030127E-05"
-        rpy="0 0 0" />
-      <mass
-        value="3.83427523968864" />
-      <inertia
-        ixx="0.0296525526652264"
-        ixy="1.5100019082583E-06"
-        ixz="2.35765651707649E-06"
-        iyy="0.0163749526901628"
-        iyz="1.22544631738128E-06"
-        izz="0.0163720507270359" />
-    </inertial>
-    <visual>
-      <origin
-        xyz="0 0 0"
-        rpy="0 0 0" />
-      <geometry>
-        <mesh
-          filename="package://ric_description/komodo/meshes/RR_Wheel_link.STL" />
-      </geometry>
-      <material
-        name="">
-        <color
-          rgba="0.15 0.15 0.15 1" />
-      </material>
-    </visual>
-    <collision>
-      <origin
-        xyz="0 0 0"
-        rpy="0 1.5 0" />
-      <geometry>
-       <!--mesh
-          filename="package://ric_description/komodo/meshes_elevator/FR_Wheel_link.STL" /-->
-        <cylinder length="0.05" radius="0.1"
-          />
-      </geometry>
-    </collision>
-  </link>
-  <joint
-    name="RR_Wheel_joint"
-    type="continuous">
-    <origin
-      xyz="-0.156000000000005 -0.2009 0"
-      rpy="2.62229105359916E-15 -1.59433090848306E-31 1.5707963267949" />
-    <parent
-      link="base_link" />
-    <child
-      link="RR_Wheel_link" />
-    <axis
-      xyz="1 0 0" />
-  </joint>
-  <link
-    name="RL_Wheel_link">
-    <inertial>
-      <origin
-        xyz="-0.00160662477936549 -2.59222765522371E-06 1.49952106412736E-05"
-        rpy="0 0 0" />
-      <mass
-        value="3.83427523542708" />
-      <inertia
-        ixx="0.0296525526119397"
-        ixy="1.5100179619978E-06"
-        ixz="2.35767335983606E-06"
-        iyy="0.0163749526769378"
-        iyz="1.22544931791974E-06"
-        izz="0.0163720506885898" />
-    </inertial>
-    <visual>
-      <origin
-        xyz="0 0 0"
-        rpy="0 0 0" />
-      <geometry>
-        <mesh
-          filename="package://ric_description/komodo/meshes/RL_Wheel_link.STL" />
-      </geometry>
-      <material
-        name="">
-        <color
-          rgba="0.15 0.15 0.15 1" />
-      </material>
-    </visual>
-    <collision>
-      <origin
-        xyz="0 0 0"
-        rpy="0 1.5 0" />
-      <geometry>
-       <!--mesh
-          filename="package://ric_description/komodo/meshes_elevator/FR_Wheel_link.STL" /-->
-        <cylinder length="0.05" radius="0.1"
-          />
-      </geometry>
-    </collision>
-  </link>
-  <joint
-    name="RL_Wheel_joint"
-    type="continuous">
-    <origin
-      xyz="-0.156000000000005 0.2009 0"
-      rpy="-2.62229105359916E-15 -5.57680208627196E-32 -1.5707963267949" />
-    <parent
-      link="base_link" />
-    <child
-      link="RL_Wheel_link" />
-    <axis
-      xyz="-1 0 0" />
-  </joint>
-  <link
-    name="Left_URF_link">
-    <inertial>
-      <origin
-        xyz="-0.00942258060476561 1.68888278492922E-05 -0.000193183712129175"
-        rpy="0 0 0" />
-      <mass
-        value="0.00277487854391404" />
-      <inertia
-        ixx="1.28314681514111E-07"
-        ixy="-1.54585356342896E-10"
-        ixz="3.11030599725484E-09"
-        iyy="1.18940672500039E-07"
-        iyz="4.35265830364889E-09"
-        izz="1.28434121553121E-07" />
-    </inertial>
-    <visual>
-      <origin
-        xyz="0 0 0"
-        rpy="0 0 0" />
-      <geometry>
-        <mesh
-          filename="package://ric_description/komodo/meshes/Left_URF_link.STL" />
-      </geometry>
-      <material
-        name="">
-        <color
-          rgba="0.752941176470588 0.752941176470588 0.752941176470588 1" />
-      </material>
-    </visual>
-    <collision>
-      <origin
-        xyz="0 0 0"
-        rpy="0 0 0" />
-      <geometry>
-        <mesh
-          filename="package://ric_description/komodo/meshes/Left_URF_link.STL" />
-      </geometry>
-    </collision>
-  </link>
-  <joint
-    name="Left_URF_joint"
-    type="fixed">
-    <origin
-      xyz="-0.0223133326154785 0.137250000000005 0.138508176066688"
-      rpy="-2.73331335606168E-15 1.59433090848306E-31 1.5707963267949" />
-    <parent
-      link="base_link" />
-    <child
-      link="Left_URF_link" />
-    <axis
-      xyz="-1 0 0" />
-  </joint>
-  <link
-    name="Rear_URF_link">
-    <inertial>
-      <origin
-        xyz="-0.00942258060476558 1.68888278491873E-05 -0.000193183712129189"
-        rpy="0 0 0" />
-      <mass
-        value="0.0027748785439141" />
-      <inertia
-        ixx="1.28314681514116E-07"
-        ixy="-1.54585356343498E-10"
-        ixz="3.1103059972555E-09"
-        iyy="1.18940672500041E-07"
-        iyz="4.35265830364838E-09"
-        izz="1.28434121553125E-07" />
-    </inertial>
-    <visual>
-      <origin
-        xyz="0 0 0"
-        rpy="0 0 0" />
-      <geometry>
-        <mesh
-          filename="package://ric_description/komodo/meshes/Rear_URF_link.STL" />
-      </geometry>
-      <material
-        name="">
-        <color
-          rgba="0.752941176470588 0.752941176470588 0.752941176470588 1" />
-      </material>
-    </visual>
-    <collision>
-      <origin
-        xyz="0 0 0"
-        rpy="0 0 0" />
-      <geometry>
-        <mesh
-          filename="package://ric_description/komodo/meshes/Rear_URF_link.STL" />
-      </geometry>
-    </collision>
-  </link>
-  <joint
-    name="Rear_URF_joint"
-    type="fixed">
-    <origin
-      xyz="-0.267499972183238 0 0.107999999999999"
-      rpy="-6.16297582203915E-33 2.73331335606168E-15 3.14159265358979" />
-    <parent
-      link="base_link" />
-    <child
-      link="Rear_URF_link" />
-    <axis
-      xyz="-1 0 0" />
-  </joint>
-  <link
-    name="Right_URF_link">
-    <inertial>
-      <origin
-        xyz="-0.00942258060476561 1.68888278493408E-05 -0.000193183712129202"
-        rpy="0 0 0" />
-      <mass
-        value="0.00277487854391409" />
-      <inertia
-        ixx="1.28314681514115E-07"
-        ixy="-1.54585356342962E-10"
-        ixz="3.11030599725548E-09"
-        iyy="1.18940672500041E-07"
-        iyz="4.3526583036484E-09"
-        izz="1.28434121553124E-07" />
-    </inertial>
-    <visual>
-      <origin
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